File: battery-charger.kicad_sch (KiCad schematic)
At the start: 12 parts, among them U4 SGM41524YTDC8G/TR

Commit message: rename project
Parts:
- removed C15: 10uF, symbol Device:C
- removed C16, C18: 100nF, symbol Device:C
- removed C17: 22uF, symbol Device:C
- removed L2: 2.2uH, symbol Device:L_Iron
- removed R13: 15K 1%, symbol Device:R
- removed R14: 20K 1%, symbol Device:R
- removed R15: 0, symbol Device:R
- removed R16: 1K, symbol Device:R
- removed TH1: 10K, symbol Device:Thermistor_NTC
- removed U4: SGM41524YTDC8G/TR, pager-jlc:DFN-8_L3.0-W2.0-P0.50-TL-EP-1, symbol pager-jlc:SGM41524YTDC8G_TR
- added C19, C20: 100nF, symbol Device:C
- added C2: 22uF, symbol Device:C
- added C6: 10uF, symbol Device:C
- added L3: 2.2uH, symbol Device:L_Iron
- added R19: 22K, symbol Device:R
- added R20: 15K, symbol Device:R
- added R22: 1K, symbol Device:R
- added TH2: 10K, symbol Device:Thermistor_NTC
- added U6: SGM41524YTDC8G/TR, pager-jlc:DFN-8_L3.0-W2.0-P0.50-TL-EP-1, symbol pager-jlc:SGM41524YTDC8G_TR
Connections:
- net +5V: now also C19.1, C6.2, R20.1, U6.7 (VIN)
- net +BATT: now also C2.2, C20.1, L3.1, U6.5 (VBAT)
- net GND: now also C19.2, C2.1, C20.2, C6.1, R19.2, R22.1, TH2.2, U6.3 (CV), U6.8 (GND), U6.9 (GND)
- net at D2.1 (K): now also R22.2
- net at D2.2 (A): now also U6.2 (IND)
- new net: R20.2, TH2.1, U6.6 (NTC)
- new net: L3.2, U6.1 (SW)
- new net: R19.1, U6.4 (CC)
Other:
- title: (none) -> Meshpager

Commit message: update
Parts:
- removed L3: 2.2uH, symbol Device:L_Iron
- added L2: 2.2uH, pager-jlc:IND-SMD_L3.0-W3.0_SWPA3010S, symbol pager-jlc:SWPA3012S2R2M
- C13: renamed from C6; footprint (none) -> Capacitor_SMD:C_0603_1608Metric
- C14: renamed from C19; footprint (none) -> Capacitor_SMD:C_0402_1005Metric
- C15: renamed from C20; footprint (none) -> Capacitor_SMD:C_0402_1005Metric
- C16: renamed from C2; footprint (none) -> Capacitor_SMD:C_0805_2012Metric
- D4: renamed from D2; footprint (none) -> LED_SMD:LED_0603_1608Metric
- R15: renamed from R20; footprint (none) -> Resistor_SMD:R_0402_1005Metric
- R16: renamed from R22; footprint (none) -> Resistor_SMD:R_0402_1005Metric
- R17: renamed from R19; footprint (none) -> Resistor_SMD:R_0402_1005Metric
- TH1: renamed from TH2; footprint (none) -> Resistor_SMD:R_0603_1608Metric
Connections:
- net +BATT: now also L2.2
- net at U6.1 (SW): now also L2.1

Commit message: update
Parts:
- removed R15: 15K, Resistor_SMD:R_0402_1005Metric, symbol Device:R
- removed TH1: 10K, Resistor_SMD:R_0603_1608Metric, symbol Device:Thermistor_NTC
- added TP14: CC, TestPoint:TestPoint_Pad_1.5x1.5mm, symbol Connector:TestPoint
- R17: value 22K -> 27K
- renumbered C13 to C19, C14 to C20, C15 to C21, C16 to C22, U6 to U5
Connections:
- net GND: now also U5.6 (NTC)
- net at R17.1, U5.4 (CC): now also TP14.1
Other:
- moved on the sheet: C19, C20, C22, D4, R16

Commit message: Update
Parts:
- TP14: footprint TestPoint:TestPoint_Pad_1.5x1.5mm -> TestPoint:TestPoint_Pad_D1.5mm; now left out of the parts list
Changed lines of the file:
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@@
 		(body_style 1)
 		(exclude_from_sim no)
-		(in_bom yes)
+		(in_bom no)
 		(on_board yes)
 		(in_pos_files yes)
@@
 			)
 		)
-		(property "Footprint" "TestPoint:TestPoint_Pad_1.5x1.5mm"
+		(property "Footprint" "TestPoint:TestPoint_Pad_D1.5mm"
 			(at 156.21 93.98 0)
 			(hide yes)

Commit message: Update
Parts:
- C19: LCSC (none) -> C19702
- C20, C21: LCSC (none) -> C1525
- C22: LCSC (none) -> C45783
- D4: LCSC (none) -> C2286
- L2: LCSC (none) -> C36402
- R16: LCSC (none) -> C11702
- R17: LCSC (none) -> C2933084
- U5: LCSC (none) -> C699852
Changed lines of the file:
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@@
+			)
+		)
+		(property "LCSC" "C1525"
+			(at 179.07 93.9799 0)
+			(hide yes)
+			(show_name no)
+			(do_not_autoplace no)
+			(effects
+				(font
+					(size 1.27 1.27)
+				)
 			)
 		)
@@
 			)
 		)
+		(property "LCSC" "C19702"
+			(at 91.44 86.3599 0)
+			(hide yes)
+			(show_name no)
+			(do_not_autoplace no)
+			(effects
+				(font
+					(size 1.27 1.27)
+				)
+			)
+		)
 		(pin "2"
 		)
@@
 			)
 		)
+		(property "LCSC" "C36402"
+			(at 165.07 72.39 0)
+			(hide yes)
+			(show_name no)
+			(do_not_autoplace no)
+			(effects
+				(font
+					(size 1.27 1.27)
+				)
+			)
+		)
 		(pin "2"
 		)
@@
 		(property "Sim.Pins" "1=K 2=A"
 			(at 115.57 87.63 0)
+			(hide yes)
+			(show_name no)
+			(do_not_autoplace no)
+			(effects
+				(font
+					(size 1.27 1.27)
+				)
+			)
+		)
+		(property "LCSC" "C2286"
+			(at 119.38 87.9474 0)
 			(hide yes)
 			(show_name no)
@@
 			)
 		)
+		(property "LCSC" "C45783"
+			(at 193.04 93.9799 0)
+			(hide yes)
+			(show_name no)
+			(do_not_autoplace no)
+			(effects
+				(font
+					(size 1.27 1.27)
+				)
+			)
+		)
 		(pin "2"
 		)
@@
 			)
 		)
+		(property "LCSC" "C2933084"
+			(at 158.75 93.9799 0)
+			(hide yes)
+			(show_name no)
+			(do_not_autoplace no)
+			(effects
+				(font
+					(size 1.27 1.27)
+				)
+			)
+		)
 		(pin "1"
 		)
@@
 		(property "Description" "Unpolarized capacitor"
 			(at 109.22 87.63 0)
+			(hide yes)
+			(show_name no)
+			(do_not_autoplace no)
+			(effects
+				(font
+					(size 1.27 1.27)
+				)
+			)
+		)
+		(property "LCSC" "C1525"
+			(at 105.41 86.3599 0)
 			(hide yes)
 			(show_name no)
@@
 			)
 		)
+		(property "LCSC" "C699852"
+			(at 146.05 71.12 0)
+			(hide yes)
+			(show_name no)
+			(do_not_autoplace no)
+			(effects
+				(font
+					(size 1.27 1.27)
+				)
+			)
+		)
 		(pin "2"
 		)
@@
 			(hide yes)
 			(show_name no)
+			(do_not_autoplace no)
+			(effects
+				(font
+					(size 1.27 1.27)
+				)
+			)
+		)
+		(property "LCSC" "C11702"
+			(at 118.11 96.5199 0)
+			(hide yes)
+			(show_name no)
