File: edp.kicad_sch (KiCad schematic)
At the start: 1 part, among them J3 B8B-PH-K-S(LF)(SN)

Commit message: update
Parts:
- removed J3: B8B-PH-K-S(LF)(SN), pager:B8BPHKSLFSN, symbol $pager:B8B-PH-K-S_LF__SN_
- added C23: 10uF, Capacitor_SMD:C_0603_1608Metric, symbol Device:C
- added J5: S8B-PH-SM4-TB, pager-jlc:CONN-SMD_8P-P2.00_S8B-PH-SM4-TB-LF-SN, symbol pager-jlc:S8B-PH-SM4-TB
Connections:
- net +3V3_S: now also C23.1, J5.1
- net EPD.BUSY: now also J5.8
- net EPD.CS: now also J5.5
- net EPD.DC: now also J5.6
- net EPD.MOSI: now also J5.3
- net EPD.RST: now also J5.7
- net EPD.SCK: now also J5.4
- net GND: now also C23.2, J5.10, J5.2, J5.9

Commit message: Update
Parts:
- C23: LCSC (none) -> C19702
- J5: LCSC (none) -> C265121
Changed lines of the file:
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@@
+			)
+		)
+		(property "LCSC" "C19702"
+			(at 148.59 120.6499 0)
+			(hide yes)
+			(show_name no)
+			(do_not_autoplace no)
+			(effects
+				(font
+					(size 1.27 1.27)
+				)
 			)
 		)
@@
 			(hide yes)
 			(show_name no)
+			(do_not_autoplace no)
+			(effects
+				(font
+					(size 1.27 1.27)
+				)
+			)
+		)
+		(property "LCSC" "C265121"
+			(at 158.75 102.8701 0)
+			(hide yes)
+			(show_name no)
