File: input_module.kicad_sch (KiCad schematic)
At the start: 14 parts, among them U8 TCA8418RTWR

Commit message: update
Parts:
- removed S7: D2F-L, pager:D2FL, symbol pager:D2F-L
- added TP15: TCA_KP_INT, TestPoint:TestPoint_Pad_1.5x1.5mm, symbol Connector:TestPoint
- added TP16: TCA_SCL, TestPoint:TestPoint_Pad_1.5x1.5mm, symbol Connector:TestPoint
- added TP17: TCA_SDA, TestPoint:TestPoint_Pad_1.5x1.5mm, symbol Connector:TestPoint
- renumbered C17 to C24, C18 to C25, U8 to U7
Connections:
- net TCA_KEYPAD_INT: now also TP15.1
- net TCA_SCL: now also TP16.1
- net TCA_SDA: now also TP17.1
- no-connect marks 14 -> 13

Commit message: Update
Parts:
- TP15, TP16, TP17: footprint TestPoint:TestPoint_Pad_1.5x1.5mm -> TestPoint:TestPoint_Pad_D1.5mm; now left out of the parts list
Changed lines of the file:
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@@
 		(body_style 1)
 		(exclude_from_sim no)
-		(in_bom yes)
+		(in_bom no)
 		(on_board yes)
 		(in_pos_files yes)
@@
 			)
 		)
-		(property "Footprint" "TestPoint:TestPoint_Pad_1.5x1.5mm"
+		(property "Footprint" "TestPoint:TestPoint_Pad_D1.5mm"
 			(at 262.89 68.58 0)
 			(hide yes)
@@
 		(body_style 1)
 		(exclude_from_sim no)
-		(in_bom yes)
+		(in_bom no)
 		(on_board yes)
 		(in_pos_files yes)
@@
 			)
 		)
-		(property "Footprint" "TestPoint:TestPoint_Pad_1.5x1.5mm"
+		(property "Footprint" "TestPoint:TestPoint_Pad_D1.5mm"
 			(at 236.22 68.58 0)
 			(hide yes)
@@
 		(body_style 1)
 		(exclude_from_sim no)
-		(in_bom yes)
+		(in_bom no)
 		(on_board yes)
 		(in_pos_files yes)
@@
 			)
 		)
-		(property "Footprint" "TestPoint:TestPoint_Pad_1.5x1.5mm"
+		(property "Footprint" "TestPoint:TestPoint_Pad_D1.5mm"
 			(at 251.46 68.58 0)
 			(hide yes)

Commit message: Pretty cool now
Parts:
- added H1, H2, H3, H4: MountingHole_Pad, MountingHole:MountingHole_2.7mm_M2.5_Pad, symbol Mechanical:MountingHole_Pad
- added TP13: GND1, TestPoint:TestPoint_Pad_D1.5mm, symbol Connector:TestPoint
- added TP3: VDD, TestPoint:TestPoint_Pad_D1.5mm, symbol Connector:TestPoint
Connections:
- net +3V3_S renamed VDD
- net VDD: now also TP3.1
- net GND renamed GND1
- net GND1: now also H1.1, H2.1, H3.1, H4.1, TP13.1

Commit message: Update
Parts:
- removed H1, H2, H3, H4: MountingHole_Pad, MountingHole:MountingHole_2.7mm_M2.5_Pad, symbol Mechanical:MountingHole_Pad
- U7: footprint pager:RTW24_2P45X2P45 -> Package_DFN_QFN:WQFN-24-1EP_4x4mm_P0.5mm_EP2.45x2.45mm

Commit message: Update
Parts:
- removed R20: 10K, Resistor_SMD:R_0805_2012Metric, symbol Device:R
- removed R23: 10K, Resistor_SMD:R_0402_1005Metric, symbol Device:R
- added RN1, RN2, RN3, RN4: R_Pack04, Resistor_SMD:R_Array_Convex_4x0603, symbol Device:R_Pack04
- C24: footprint Capacitor_SMD:C_0805_2012Metric -> Capacitor_SMD:C_0402_1005Metric; LCSC (none) -> C1525
- C25: footprint Capacitor_SMD:C_0805_2012Metric -> Capacitor_SMD:C_0603_1608Metric; LCSC (none) -> C15849
- R21, R22: LCSC (none) -> C25744
- S1, S2, S3, S4, S5, S6: LCSC (none) -> C231329
- U7: LCSC (none) -> C138713
Connections:
- net TCA_KEYPAD_INT: now also RN2.3 (R3.1)
- net VDD: now also RN1.5 (R4.2), RN1.6 (R3.2), RN1.7 (R2.2), RN1.8 (R1.2), RN2.6 (R3.2), RN2.7 (R2.2), RN2.8 (R1.2), RN3.1 (R1.1), RN3.2 (R2.1), RN3.3 (R3.1), RN3.4 (R4.1), RN4.1 (R1.1), RN4.2 (R2.1), RN4.3 (R3.1), RN4.4 (R4.1)
- net at U7.20 (*RESET): now also RN4.5 (R4.2)
- net at U7.1 (ROW7): now also RN2.2 (R2.1)
- net at U7.12 (COL3): now also RN3.8 (R1.2)
- net at U7.13 (COL4): now also RN3.7 (R2.2)
- net at U7.14 (COL5): now also RN3.6 (R3.2)
- net at U7.15 (COL6): now also RN3.5 (R4.2)
- net at U7.16 (COL7): now also RN4.8 (R1.2)
- net at U7.17 (COL8): now also RN4.7 (R2.2)
- net at U7.18 (COL9): now also RN4.6 (R3.2)
- net at U7.2 (ROW6): now also RN2.1 (R1.1)
- net at U7.3 (ROW5): now also RN1.4 (R4.1)
- net at U7.4 (ROW4): now also RN1.3 (R3.1)
- net at U7.5 (ROW3): now also RN1.2 (R2.1)
- net at U7.6 (ROW2): now also RN1.1 (R1.1)
- no-connect marks 13 -> 2
