File: mcu.kicad_sch (KiCad schematic)
At the start: 11 parts, among them J1 Conn_01x05, SW2 SW_SPST, U4 RAK4630-8-SM-I

Commit message: update
Parts:
- removed R15, R16: 10K, symbol Device:R
- C1: renamed from C15; value C -> 100nF; footprint (none) -> Capacitor_SMD:C_0402_1005Metric
- D1: renamed from D3; footprint (none) -> LED_SMD:LED_0603_1608Metric
- D2: renamed from D4; footprint (none) -> LED_SMD:LED_0603_1608Metric
- J1: footprint (none) -> Connector_PinHeader_1.27mm:PinHeader_1x05_P1.27mm_Vertical_SMD_Pin1Left; now not fitted; now left out of the parts list
- R1: renamed from R21; footprint (none) -> Resistor_SMD:R_0402_1005Metric
- R2: renamed from R5; footprint (none) -> Resistor_SMD:R_0402_1005Metric
- R3: renamed from R13; footprint (none) -> Resistor_SMD:R_0402_1005Metric
- SW1: renamed from SW2; footprint (none) -> pager:B3U-1000P
- renumbered U4 to U1
Connections:
- net I2C1.SCL: now also U1.5 (P0.14/12C_SCL); no longer U1.4 (P0.13/12C_SDA)
- net I2C1.SDA: now also U1.4 (P0.13/12C_SDA); no longer U1.5 (P0.14/12C_SCL)
- net +3.3V renamed +3V3
- net EPD.DC_* renamed EPD.DC
- net EPD.RST_* renamed EPD.RST
Other:
- moved on the sheet: D1, D2, R2, R3

Commit message: update
Parts:
- added C2, C3: 100nF, Capacitor_SMD:C_0402_1005Metric, symbol Device:C
- added C4: 10uF, Capacitor_SMD:C_0603_1608Metric, symbol Device:C
- added J2: Conn_01x03, Connector_PinHeader_1.27mm:PinHeader_1x03_P1.27mm_Vertical_SMD_Pin1Left, symbol Connector_Generic:Conn_01x03
Connections:
- net +3V3: now also C2.1, C3.1, C4.1
- net GND: now also C2.2, C3.2, C4.2, J2.3 (Pin_3)
- net UART1_TX: now reaches U1.10 (P0.20/UART1_TX)
- net UART1_TX: now also J2.1 (Pin_1)
- net UART1_RX: now reaches U1.9 (P0.19/UART1_RX)
- net UART1_RX: now also J2.2 (Pin_2)
- net SW1: no longer names the net of U1.25 (P1.01/SW1)
- no-connect marks 13 -> 12

Commit message: Update
Parts:
- C1, C2, C3: LCSC (none) -> C1525
- C4: LCSC (none) -> C19702
- D1: value LED -> GREEN; LCSC (none) -> C12624
- D2: value LED -> BLUE; LCSC (none) -> C2288
- J1: footprint Connector_PinHeader_1.27mm:PinHeader_1x05_P1.27mm_Vertical_SMD_Pin1Left -> Connector_PinHeader_1.27mm:PinHeader_1x05_P1.27mm_Vertical
- J2: footprint Connector_PinHeader_1.27mm:PinHeader_1x03_P1.27mm_Vertical_SMD_Pin1Left -> Connector_PinHeader_1.27mm:PinHeader_1x03_P1.27mm_Vertical
- R1: LCSC (none) -> C25744
- R2, R3: LCSC (none) -> C11702
- SW1: value SW_SPST -> B3U-1000P; LCSC (none) -> C231329
- U1: LCSC (none) -> C32315253
Changed lines of the file:
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@@
+			)
+		)
+		(property "LCSC" "C25744"
+			(at 38.1 147.3199 0)
+			(hide yes)
+			(show_name no)
+			(do_not_autoplace no)
+			(effects
+				(font
+					(size 1.27 1.27)
+				)
 			)
 		)
@@
 			)
 		)
+		(property "LCSC" "C1525"
+			(at 34.29 161.2899 0)
+			(hide yes)
+			(show_name no)
+			(do_not_autoplace no)
+			(effects
+				(font
+					(size 1.27 1.27)
+				)
+			)
+		)
 		(pin "1"
 		)
@@
 			)
 		)
-		(property "Value" "LED"
+		(property "Value" "GREEN"
 			(at 207.01 117.1574 90)
 			(show_name no)
@@
 			)
 		)
+		(property "LCSC" "C12624"
+			(at 207.01 114.6174 0)
+			(hide yes)
+			(show_name no)
+			(do_not_autoplace no)
+			(effects
+				(font
+					(size 1.27 1.27)
+				)
+			)
+		)
 		(pin "2"
 		)
@@
 			)
 		)
-		(property "Value" "LED"
+		(property "Value" "BLUE"
 			(at 217.17 117.1574 90)
 			(show_name no)
@@
 			)
 		)
+		(property "LCSC" "C2288"
+			(at 217.17 114.6174 0)
+			(hide yes)
+			(show_name no)
+			(do_not_autoplace no)
+			(effects
+				(font
+					(size 1.27 1.27)
+				)
+			)
+		)
 		(pin "2"
 		)
@@
 			)
 		)
+		(property "LCSC" "C19702"
+			(at 193.04 41.9099 0)
+			(hide yes)
+			(show_name no)
+			(do_not_autoplace no)
+			(effects
+				(font
+					(size 1.27 1.27)
+				)
+			)
+		)
 		(pin "1"
 		)
@@
 			)
 		)
+		(property "LCSC" "C1525"
+			(at 233.68 41.9099 0)
+			(hide yes)
+			(show_name no)
+			(do_not_autoplace no)
+			(effects
+				(font
+					(size 1.27 1.27)
+				)
+			)
+		)
 		(pin "1"
 		)
@@
 			)
 		)
-		(property "Footprint" "Connector_PinHeader_1.27mm:PinHeader_1x03_P1.27mm_Vertical_SMD_Pin1Left"
+		(property "Footprint" "Connector_PinHeader_1.27mm:PinHeader_1x03_P1.27mm_Vertical"
 			(at 149.86 149.86 0)
 			(hide yes)
@@
 			)
 		)
-		(property "Value" "SW_SPST"
+		(property "Value" "B3U-1000P"
 			(at 43.18 163.8299 90)
 			(show_name no)
@@
 			)
 		)
+		(property "LCSC" "C231329"
+			(at 43.18 161.2899 0)
+			(hide yes)
+			(show_name no)
+			(do_not_autoplace no)
+			(effects
+				(font
+					(size 1.27 1.27)
+				)
+			)
+		)
 		(pin "2"
 		)
@@
 			)
 		)
-		(property "Footprint" "Connector_PinHeader_1.27mm:PinHeader_1x05_P1.27mm_Vertical_SMD_Pin1Left"
+		(property "Footprint" "Connector_PinHeader_1.27mm:PinHeader_1x05_P1.27mm_Vertical"
 			(at 107.95 149.86 0)
 			(hide yes)
@@
 			)
 		)
+		(property "LCSC" "C32315253"
+			(at 143.51 52.07 0)
+			(hide yes)
+			(show_name no)
+			(do_not_autoplace no)
+			(effects
+				(font
+					(size 1.27 1.27)
+				)
+			)
+		)
 		(pin "12"
 		)
@@
 			)
 		)
+		(property "LCSC" "C11702"
+			(at 205.74 124.4599 0)
+			(hide yes)
+			(show_name no)
+			(do_not_autoplace no)
+			(effects
+				(font
+					(size 1.27 1.27)
+				)
+			)
+		)
 		(pin "2"
 		)
@@
 			)
 		)
+		(property "LCSC" "C1525"
+			(at 260.35 43.1799 0)
+			(hide yes)
+			(show_name no)
+			(do_not_autoplace no)
+			(effects
+				(font
+					(size 1.27 1.27)
+				)
+			)
+		)
 		(pin "1"
 		)
@@
 			(hide yes)
 			(show_name no)
+			(do_not_autoplace no)
+			(effects
+				(font
+					(size 1.27 1.27)
+				)
+			)
+		)
+		(property "LCSC" "C11702"
+			(at 215.9 124.4599 0)
+			(hide yes)
+			(show_name no)
