File: meshpager.kicad_pcb (KiCad board)
At the start: 2 copper layers, 92 x 66 mm, 75 parts, among them J1 Conn_01x05, J2 USB_C_Receptacle_USB2.0_16P, J3 B8B-PH-K-S(LF)(SN), Q1 NCE40P05Y, SW1 SW_SPST, SW2 MK-12C02-G020, U1 RAK4630-8-SM-I, U2 GT-BTP30003-0600A-016A, U3 SGM2578AADYG/TR, U4 SGM6036-3.3YUDT6G/TR, U5 SY6287CABC, U6 SGM41524YTDC8G/TR, U7 USBLC6-2SC6, U8 TCA8418RTWR

Commit message: update
Parts:
- removed C1, C11, C14, C15, C2, C3, C6, C7, C8, C9: 100nF, Capacitor_SMD:C_0402_1005Metric
- removed C10, C16, C4: 22uF, Capacitor_SMD:C_0805_2012Metric
- removed C12, C13, C5: 10uF, Capacitor_SMD:C_0603_1608Metric
- removed C17: 100nF, Capacitor_SMD:C_0805_2012Metric
- removed C18: 1uF, Capacitor_SMD:C_0805_2012Metric
- removed D1, D2: LED, LED_SMD:LED_0603_1608Metric
- removed D3: MBR140SFT1G, pager-jlc:SOD-123F_L2.8-W1.8-LS3.7-RD
- removed D4: RED, LED_SMD:LED_0603_1608Metric
- removed H5, H6: MountingHole_Pad, MountingHole:MountingHole_2.7mm_M2.5_Pad
- removed J1: Conn_01x05, Connector_PinHeader_1.27mm:PinHeader_1x05_P1.27mm_Vertical_SMD_Pin1Left
- removed J2: USB_C_Receptacle_USB2.0_16P, Connector_USB:USB_C_Receptacle_HRO_TYPE-C-31-M-12
- removed L1: 4.7uH, pager-jlc:IND-SMD_L3.0-W3.0_FNR30XXS
- removed L2: 2.2uH, pager-jlc:IND-SMD_L3.0-W3.0_SWPA3010S
- removed Q1: NCE40P05Y, pager-jlc:SOT-23-3_L2.9-W1.6-P1.90-LS2.8-BR
- removed R1, R21, R22, R23, R7: 10K, Resistor_SMD:R_0402_1005Metric
- removed R10, R9: 4.7K, Resistor_SMD:R_0402_1005Metric
- removed R11, R8: 100K, Resistor_SMD:R_0402_1005Metric
- removed R12, R14, R6: 0, Resistor_SMD:R_0402_1005Metric
- removed R13: 470 1%, Resistor_SMD:R_0402_1005Metric
- removed R15: 15K, Resistor_SMD:R_0402_1005Metric
- removed R16, R2, R3: 1K, Resistor_SMD:R_0402_1005Metric
- removed R17: 22K, Resistor_SMD:R_0402_1005Metric
- removed R18, R19: 5.1K, Resistor_SMD:R_0402_1005Metric
- removed R20: 10K, Resistor_SMD:R_0805_2012Metric
- removed R4: 1M, Resistor_SMD:R_0402_1005Metric
- removed R5: 1.5M, Resistor_SMD:R_0402_1005Metric
- removed S7: D2F-L, pager:D2FL
- removed SW1: SW_SPST, pager:B3U-1000P
- removed SW2: MK-12C02-G020, pager-jlc:SW-SMD_MK-12C02-G020
- removed TH1: 10K, Resistor_SMD:R_0603_1608Metric
- removed U2: GT-BTP30003-0600A-016A, pager-jlc:BAT-SMD_GT-BTP30003-0500A-016A-1
- removed U3: SGM2578AADYG/TR, pager-jlc:WLCSP-4_L0.9-W0.9-R2-C2-P0.50-TL
- removed U4: SGM6036-3.3YUDT6G/TR, pager-jlc:UTDFN-6_L2.0-W1.5-P0.50-BL-EP
- removed U5: SY6287CABC, pager-jlc:SOT-23-6_L2.9-W1.6-P0.95-LS2.9-BL
- removed U6: SGM41524YTDC8G/TR, pager-jlc:DFN-8_L3.0-W2.0-P0.50-TL-EP-1
- removed U7: USBLC6-2SC6, Package_TO_SOT_SMD:SOT-23-6
- removed U8: TCA8418RTWR, pager:RTW24_2P45X2P45
- added J4: USB_C_Receptacle_USB2.0_16P, Connector_USB:USB_C_Receptacle_G-Switch_GT-USB-7010ASV, F.Cu at (186.8, 95.3)
- added J5: S8B-PH-SM4-TB, pager-jlc:CONN-SMD_8P-P2.00_S8B-PH-SM4-TB-LF-SN, F.Cu at (120.1, 70.5)
- J3: value B8B-PH-K-S(LF)(SN) -> 009155003301006; footprint pager:B8BPHKSLFSN -> pager:009155003301006; moved to B.Cu
- moved J3 122.2 mm to (119.3, 86.3), turned to 90 degrees
- moved U1 117.8 mm to (145.0, 85.0)
- moved H4 76.8 mm to (182.9, 85.7)
- moved H2 56.8 mm to (182.9, 54.4)
- moved H1 55.7 mm to (105.1, 54.4)
- moved H3 47.7 mm to (105.1, 85.7)
- moved S3 7.57 mm to (168.5, 101.2), turned to 0 degrees
- moved S2 5.59 mm to (168.5, 107.8), turned to 0 degrees
- moved S1 1.41 mm to (179.9, 104.5), turned to 0 degrees
- moved S4 1.41 mm to (157.1, 104.5), turned to 0 degrees
- moved S5 1.41 mm to (128.1, 98.2), turned to 0 degrees
- moved S6 1.41 mm to (112.8, 98.2), turned to 0 degrees
Connections:
- J3 pad 1: +3V3_S -> GND
- J3 pad 2: GND -> unconnected-(J3-Pad2)
- J3 pad 3: /edp/EPD.MOSI -> unconnected-(J3-Pad3)
- J3 pad 4: /edp/EPD.SCK -> unconnected-(J3-Pad4)
- J3 pad 5: /edp/EPD.CS -> BAT_CELL
- J3 pad 6: /edp/EPD.DC -> unconnected-(J3-Pad6)
- J3 pad 7: /edp/EPD.RST -> unconnected-(J3-Pad7)
- U1 pad 10: unconnected-(U1-P0.20/UART1_TX-Pad10) -> /mcu/UART1_TX
- U1 pad 25: /input_module/SW1 -> unconnected-(U1-P1.01/SW1-Pad25)
- U1 pad 9: unconnected-(U1-P0.19/UART1_RX-Pad9) -> /mcu/UART1_RX
Routing:
- added copper zone on B.Cu, net GND
- added copper zone on F.Cu, net GND
- added copper zone on In1.Cu, net GND
- added copper zone on In2.Cu, net GND
Other:
- board size 92 x 66 mm -> 90 x 64 mm
- copper layers 2 -> 4

Commit message: Update
Parts:
- added C1: 100nF, Capacitor_SMD:C_0402_1005Metric, F.Cu at (72.2, 79.5)
- added C10: 10uF, Capacitor_SMD:C_0603_1608Metric, F.Cu at (64.0, 106.2)
- added C11: 100nF, Capacitor_SMD:C_0402_1005Metric, F.Cu at (62.2, 106.5)
- added C12: 22uF, Capacitor_SMD:C_0805_2012Metric, F.Cu at (49.0, 57.5)
- added C13: 100nF, Capacitor_SMD:C_0402_1005Metric, F.Cu at (64.4, 111.8)
- added C14: 100nF, Capacitor_SMD:C_0402_1005Metric, F.Cu at (45.5, 56.2)
- added C15: 100nF, Capacitor_SMD:C_0402_1005Metric, F.Cu at (44.3, 54.0)
- added C16: 22uF, Capacitor_SMD:C_0805_2012Metric, F.Cu at (50.3, 52.8)
- added C17: 100nF, Capacitor_SMD:C_0402_1005Metric, F.Cu at (54.2, 52.8)
- added C18: 10uF, Capacitor_SMD:C_0603_1608Metric, F.Cu at (69.8, 107.0)
- added C19: 10uF, Capacitor_SMD:C_0603_1608Metric, F.Cu at (65.0, 70.0)
- added C2: 100nF, Capacitor_SMD:C_0402_1005Metric, F.Cu at (38.2, 91.3)
- added C20: 100nF, Capacitor_SMD:C_0402_1005Metric, F.Cu at (61.8, 68.5)
- added C21: 100nF, Capacitor_SMD:C_0402_1005Metric, F.Cu at (54.2, 68.8)
- added C22: 22uF, Capacitor_SMD:C_0805_2012Metric, F.Cu at (57.2, 69.2)
- added C23: 10uF, Capacitor_SMD:C_0603_1608Metric, F.Cu at (39.2, 54.5)
- added C24: 100nF, Capacitor_SMD:C_0805_2012Metric, F.Cu at (145.8, 84.5)
- added C25: 1uF, Capacitor_SMD:C_0805_2012Metric, F.Cu at (145.8, 82.2)
- added C3: 100nF, Capacitor_SMD:C_0402_1005Metric, F.Cu at (39.5, 91.3)
- added C4: 10uF, Capacitor_SMD:C_0603_1608Metric, F.Cu at (36.8, 91.0)
- added C5: 100nF, Capacitor_SMD:C_0402_1005Metric, F.Cu at (62.0, 53.5)
- added C6: 100nF, Capacitor_SMD:C_0402_1005Metric, F.Cu at (38.8, 85.3)
- added C7: 10uF, Capacitor_SMD:C_0603_1608Metric, F.Cu at (62.0, 56.8)
- added C8: 1uF, Capacitor_SMD:C_0603_1608Metric, F.Cu at (67.8, 53.2)
- added C9: 100nF, Capacitor_SMD:C_0402_1005Metric, F.Cu at (70.8, 71.8)
- added D1: LED, LED_SMD:LED_0603_1608Metric, F.Cu at (34.2, 108.8)
- added D2: LED, LED_SMD:LED_0603_1608Metric, F.Cu at (34.2, 111.8)
- added D3: MBR140SFT1G, pager-jlc:SOD-123F_L2.8-W1.8-LS3.7-RD, F.Cu at (70.8, 74.8)
- added D4: RED, LED_SMD:LED_0603_1608Metric, F.Cu at (34.2, 105.8)
- added J1: Conn_01x05, Connector_PinHeader_1.27mm:PinHeader_1x05_P1.27mm_Vertical_SMD_Pin1Left, F.Cu at (72.0, 86.0)
- added J2: Conn_01x03, Connector_PinHeader_1.27mm:PinHeader_1x03_P1.27mm_Vertical_SMD_Pin1Left, F.Cu at (57.8, 100.5)
- added L1: 4.7uH, pager-jlc:IND-SMD_L3.0-W3.0_FNR30XXS, F.Cu at (53.8, 57.5)
- added L2: 2.2uH, pager-jlc:IND-SMD_L3.0-W3.0_SWPA3010S, F.Cu at (54.2, 64.7)
- added Q1: NCE40P05Y, pager-jlc:SOT-23-3_L2.9-W1.6-P1.90-LS2.8-BR, F.Cu at (70.8, 67.8)
- added R1: 10K, Resistor_SMD:R_0402_1005Metric, F.Cu at (72.2, 78.2)
- added R10: 100K, Resistor_SMD:R_0402_1005Metric, F.Cu at (62.9, 111.8)
- added R11: 100K, Resistor_SMD:R_0402_1005Metric, F.Cu at (45.5, 54.0)
- added R12: 0, Resistor_SMD:R_0805_2012Metric_Pad1.20x1.40mm_HandSolder, F.Cu at (67.4, 106.7)
- added R13: 470 1%, Resistor_SMD:R_0402_1005Metric, F.Cu at (71.9, 111.7)
- added R14: 0, Resistor_SMD:R_0805_2012Metric_Pad1.20x1.40mm_HandSolder, F.Cu at (71.9, 115.8)
- added R16: 1K, Resistor_SMD:R_0402_1005Metric, F.Cu at (34.0, 104.2)
- added R17: 27K, Resistor_SMD:R_0402_1005Metric, F.Cu at (59.5, 64.8)
- added R18: 5.1K, Resistor_SMD:R_0402_1005Metric, F.Cu at (47.2, 121.5)
- added R19: 5.1K, Resistor_SMD:R_0402_1005Metric, F.Cu at (60.8, 121.5)
- added R2: 1K, Resistor_SMD:R_0402_1005Metric, F.Cu at (34.0, 107.2)
- added R20: 10K, Resistor_SMD:R_0805_2012Metric, F.Cu at (145.8, 86.8)
- added R21: 10K, Resistor_SMD:R_0402_1005Metric, F.Cu at (142.8, 84.5)
- added R22: 10K, Resistor_SMD:R_0402_1005Metric, F.Cu at (142.8, 86.8)
- added R23: 10K, Resistor_SMD:R_0402_1005Metric, F.Cu at (142.7, 82.2)
- added R3: 1K, Resistor_SMD:R_0402_1005Metric, F.Cu at (34.0, 110.2)
- added R4: 1M, Resistor_SMD:R_0402_1005Metric, F.Cu at (40.0, 83.3)
- added R5: 1.5M, Resistor_SMD:R_0402_1005Metric, F.Cu at (40.0, 85.3)
- added R6: 0, Resistor_SMD:R_0805_2012Metric_Pad1.20x1.40mm_HandSolder, F.Cu at (65.0, 54.0)
- added R7: 4.7K, Resistor_SMD:R_0402_1005Metric, F.Cu at (68.5, 68.5)
- added R8: 10K, Resistor_SMD:R_0402_1005Metric, F.Cu at (67.5, 58.5)
- added R9: 100K, Resistor_SMD:R_0402_1005Metric, F.Cu at (69.0, 58.5)
- added SW1: SW_SPST, pager:B3U-1000P, F.Cu at (72.2, 81.2)
- added SW2: MK-12C02-G020, pager-jlc:SW-SMD_MK-12C02-G020, B.Cu at (71.5, 55.5)
- added TP1: GND, TestPoint:TestPoint_Pad_D1.5mm, F.Cu at (34.5, 52.2)
- added TP10: +3V3, TestPoint:TestPoint_Pad_D1.5mm, F.Cu at (33.8, 96.0)
- added TP11: +3V3_S, TestPoint:TestPoint_Pad_D1.5mm, F.Cu at (57.8, 54.0)
- added TP12: +BATT, TestPoint:TestPoint_Pad_D1.5mm, F.Cu at (36.0, 81.5)
- added TP14: CC, TestPoint:TestPoint_Pad_D1.5mm, F.Cu at (57.5, 64.2)
- added TP15: TCA_KP_INT, TestPoint:TestPoint_Pad_D1.5mm, F.Cu at (54.0, 99.0)
- added TP16: TCA_SCL, TestPoint:TestPoint_Pad_D1.5mm, F.Cu at (54.0, 102.0)
- added TP17: TCA_SDA, TestPoint:TestPoint_Pad_D1.5mm, F.Cu at (49.8, 102.8)
- added TP2: GND, TestPoint:TestPoint_Pad_D1.5mm, F.Cu at (61.5, 97.2)
- added TP3: GND, TestPoint:TestPoint_Pad_D1.5mm, F.Cu at (26.8, 71.0)
- added TP4: GND, TestPoint:TestPoint_Pad_D1.5mm, F.Cu at (36.0, 119.8)
- added TP5: VBAT_ADC, TestPoint:TestPoint_Pad_D1.5mm, F.Cu at (36.0, 87.0)
- added TP6: VBUS, TestPoint:TestPoint_Pad_D1.5mm, F.Cu at (41.2, 96.0)
- added TP7: +5V, TestPoint:TestPoint_Pad_D1.5mm, F.Cu at (68.8, 95.8)
- added TP8: VDC, TestPoint:TestPoint_Pad_D1.5mm, F.Cu at (73.8, 64.0)
- added TP9: MCU_GATE, TestPoint:TestPoint_Pad_D1.5mm, F.Cu at (70.0, 55.5)
- added U2: SGM2578AADYG/TR, pager-jlc:WLCSP-4_L0.9-W0.9-R2-C2-P0.50-TL, F.Cu at (65.0, 57.0)
- added U3: SY6287CABC, pager-jlc:SOT-23-6_L2.9-W1.6-P0.95-LS2.9-BL, F.Cu at (66.9, 111.2)
- added U4: SGM6036-3.3YUDT6G/TR, pager-jlc:UTDFN-6_L2.0-W1.5-P0.50-BL-EP, F.Cu at (49.0, 55.4)
- added U5: SGM41524YTDC8G/TR, pager-jlc:DFN-8_L3.0-W2.0-P0.50-TL-EP-1, F.Cu at (61.5, 65.5)
- added U6: USBLC6-2SC6, Package_TO_SOT_SMD:SOT-23-6, F.Cu at (54.8, 114.8)
- added U7: TCA8418RTWR, pager:RTW24_2P45X2P45, F.Cu at (145.3, 92.8)
- moved J4 135.6 mm to (54.0, 122.5), turned to 0 degrees
- moved U1 91.0 mm to (54.0, 86.5), turned to 180 degrees
- moved J5 79.2 mm to (41.0, 67.2)
- moved J3 62.4 mm to (62.6, 60.0), turned to 0 degrees
Routing:
- net +3V3: track 0.00 -> 114.7 mm, vias 0 -> 2
- net VBUS: track 0.00 -> 80.1 mm, vias 0 -> 5
- net +BATT: track 0.00 -> 78.5 mm, vias 0 -> 3
- net +5V: track 0.00 -> 67.7 mm, vias 0 -> 3
- net Net-(D4-A): track 0.00 -> 56.9 mm, vias 0 -> 2
- net +3V3_S: track 0.00 -> 52.8 mm, vias 0 -> 2
- net VDC: track 0.00 -> 51.5 mm, vias 0 -> 1
- net Net-(D2-A): track 0.00 -> 46.2 mm, vias 0 -> 2
- net Net-(D1-A): track 0.00 -> 45.0 mm, vias 0 -> 2
- net /mcu/USB_P: track 0.00 -> 23.1 mm
- net /mcu/USB_N: track 0.00 -> 23.1 mm
- net /mcu/NRF_RESET: track 0.00 -> 20.4 mm
- net /edp/EPD.MOSI: track 0.00 -> 20.0 mm, vias 0 -> 2
- net /input_module/TCA_SCL: track 0.00 -> 20.0 mm, vias 0 -> 2
- net /edp/EPD.SCK: track 0.00 -> 19.6 mm
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Other:
- board size 90 x 64 mm -> 160 x 79 mm
- board text added: "LEDS/SW"

Commit message: Pretty cool now
Parts:
- removed H1, H2: MountingHole_Pad, MountingHole:MountingHole_2.7mm_M2.5_Pad
- added J6: HC-FPC-05-09-5RLTAG, pager-jlc:CONN-SMD_5P-P0.50_HCTL_HC-FPC-05-09-5RLTAG, F.Cu at (120.8, 89.5)
- added J7: HC-FPC-05-09-5RLTAG, pager-jlc:CONN-SMD_5P-P0.50_HCTL_HC-FPC-05-09-5RLTAG, F.Cu at (53.2, 99.0)
- added TP13: GND1, TestPoint:TestPoint_Pad_D1.5mm, B.Cu at (139.8, 100.8)
- TP15, TP16, TP17: moved to B.Cu
- TP3: value GND -> VDD; moved to B.Cu
- moved TP3 120.9 mm to (146.2, 89.5), turned to 180 degrees
- moved TP17 90.3 mm to (139.8, 95.2), turned to 180 degrees
- moved TP15 86.0 mm to (139.8, 92.8), turned to 180 degrees
- moved TP16 85.8 mm to (139.8, 98.0), turned to 180 degrees
- moved J2 19.8 mm to (66.5, 118.2), turned to 0 degrees
- moved U7 11.2 mm to (144.8, 104.0)
- moved R23 10.0 mm to (142.0, 92.2), turned to -90 degrees
- moved C24 9.62 mm to (147.2, 94.0)
- moved C25 9.62 mm to (147.2, 91.8)
- moved R20 9.62 mm to (147.2, 96.2)
- moved R21 7.77 mm to (143.2, 92.2), turned to -90 degrees
- moved R22 5.77 mm to (144.5, 92.2), turned to -90 degrees
Connections:
- C24 pad 1: +3V3_S -> VDD
- C24 pad 2: GND -> GND1
- C25 pad 1: +3V3_S -> VDD
- C25 pad 2: GND -> GND1
- H3 pad 1: GND -> GND1
- H4 pad 1: GND -> GND1
- R20 pad 1: +3V3_S -> VDD
- R21 pad 1: +3V3_S -> VDD
- R22 pad 1: +3V3_S -> VDD
- R23 pad 1: +3V3_S -> VDD
- TP3 pad 1: GND -> VDD
- U1 pad 4: /input_module/TCA_SDA -> /mcu/I2C1.SDA
- U1 pad 5: /input_module/TCA_SCL -> /mcu/I2C1.SCL
- U1 pad 8: /input_module/TCA_KEYPAD_INT -> /mcu/KBD_INT
- U7 pad 19: GND -> GND1
- U7 pad 21: +3V3_S -> VDD
- U7 pad 25: GND -> GND1
- U7 pad V: GND -> GND1
Routing:
- net Net-(S1-K): track 0.00 -> 81.8 mm
- net Net-(S2-K): track 0.00 -> 74.5 mm, vias 0 -> 2
- net Net-(S5-A): track 0.00 -> 54.4 mm, vias 0 -> 2
- net VDD: track 0.00 -> 44.3 mm, vias 0 -> 1
- net Net-(S1-A): track 0.00 -> 40.1 mm
- net +3V3_S: track 52.8 -> 82.0 mm, vias 2 -> 3
- net Net-(S3-A): track 0.00 -> 27.2 mm
- net /mcu/UART1_RX: track 8.97 -> 32.7 mm
- net /mcu/UART1_TX: track 6.00 -> 27.9 mm
- net /input_module/TCA_SDA: track 15.8 -> 35.3 mm
- net /input_module/TCA_SCL: track 20.0 -> 36.8 mm
- net /input_module/TCA_KEYPAD_INT: track 19.5 -> 31.7 mm, vias 2 -> 1
- net /mcu/KBD_INT: track 0.00 -> 10.2 mm
- net /mcu/IO2: track 17.3 -> 25.5 mm, vias 1 -> 2
- net /mcu/I2C1.SDA: track 0.00 -> 6.93 mm
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- added copper zone on B.Cu, net GND1
- added copper zone on F.Cu, net GND1
- added copper zone on In1.Cu, net GND1
- added copper zone on In2.Cu, net GND1
Other:
- outline, holes or cut-outs redrawn

Commit message: Update
Parts:
- removed H3, H4: MountingHole_Pad, MountingHole:MountingHole_2.7mm_M2.5_Pad
- added FID1: Fiducial, Fiducial:Fiducial_1mm_Mask3mm, F.Cu at (104.0, 124.0)
- added FID2: Fiducial, Fiducial:Fiducial_1mm_Mask3mm, F.Cu at (144.0, 54.0)
- added FID3: Fiducial, Fiducial:Fiducial_1mm_Mask3mm, F.Cu at (104.0, 54.0)
- added FID4: Fiducial, Fiducial:Fiducial_1mm_Mask3mm, F.Cu at (160.0, 130.0)
- added FID5: Fiducial, Fiducial:Fiducial_1mm_Mask3mm, F.Cu at (160.0, 48.0)
- added FID6: Fiducial, Fiducial:Fiducial_1mm_Mask3mm, F.Cu at (178.0, 130.0)
- added H5: MountingHole_Pad, MountingHole:MountingHole_2.7mm_M2.5_Pad, F.Cu at (104.0, 59.0)
- added H6: MountingHole_Pad, MountingHole:MountingHole_2.7mm_M2.5_Pad, F.Cu at (144.0, 59.0)
- added H7: MountingHole_Pad, MountingHole:MountingHole_2.7mm_M2.5_Pad, F.Cu at (104.0, 118.5)
- added H8: MountingHole_Pad, MountingHole:MountingHole_2.7mm_M2.5_Pad, F.Cu at (144.0, 118.5)
- added Input: Board, PCM_kikit:Board, F.Cu at (166.8, 44.0)
- added Main: Board, PCM_kikit:Board, F.Cu at (103.8, 50.0)
- U7: footprint pager:RTW24_2P45X2P45 -> Package_DFN_QFN:WQFN-24-1EP_4x4mm_P0.5mm_EP2.45x2.45mm
- moved TP4 77.1 mm to (113.0, 116.0)
- moved J5 72.3 mm to (113.2, 70.5)
- moved S6 72.1 mm to (171.8, 56.8), turned to -90 degrees
- moved R14 71.9 mm to (143.8, 113.0), turned to 90 degrees
- moved TP1 71.3 mm to (104.0, 68.0)
- moved C23 70.3 mm to (109.5, 56.5)
- moved C16 70.2 mm to (120.5, 54.5)
- moved C9 70.0 mm to (140.8, 73.8)
- moved D3 70.0 mm to (140.8, 76.8)
- moved R1 70.0 mm to (142.2, 80.2)
- moved C1 70.0 mm to (142.2, 81.5)
- moved C10 70.0 mm to (134.0, 108.2)
- moved C11 70.0 mm to (132.2, 108.5)
- moved C12 70.0 mm to (119.0, 59.5)
- moved C13 70.0 mm to (134.4, 113.8)
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Routing:
- net BAT_CELL: track 8.66 -> 30.5 mm
- net /input_module/TCA_KEYPAD_INT: track 31.7 -> 14.4 mm
- net +3V3_S: track 82.0 -> 97.9 mm
- net /input_module/TCA_SCL: track 36.8 -> 20.9 mm
- net /input_module/TCA_SDA: track 35.3 -> 21.1 mm
- net VDD: track 44.3 -> 35.8 mm
- net /mcu/IO2: track 25.5 -> 33.5 mm
- net +BATT: track 78.5 -> 82.8 mm, vias 5 -> 4
- net Net-(U7-*RESET): track 6.88 -> 3.01 mm
- net GND: track 11.4 -> 8.26 mm, vias 16 -> 15
- net /edp/EPD.SCK: track 19.6 -> 16.8 mm
- net /edp/EPD.RST: track 15.2 -> 12.4 mm
- net Net-(D1-A): track 42.1 -> 40.3 mm
- net /edp/EPD.DC: track 14.2 -> 15.8 mm
- net Net-(U2-ON): track 6.67 -> 8.08 mm
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Other:
- board size 160 x 79 mm -> 82.5 x 90 mm
- board text removed: "LEDS/SW"

Commit message: Update
Parts:
- removed R20: 10K, Resistor_SMD:R_0805_2012Metric
- removed R23: 10K, Resistor_SMD:R_0402_1005Metric
- removed R6: 0, Resistor_SMD:R_0805_2012Metric_Pad1.20x1.40mm_HandSolder
- removed U2: SGM2578AADYG/TR, pager-jlc:WLCSP-4_L0.9-W0.9-R2-C2-P0.50-TL
- added C26: 1nF, Capacitor_SMD:C_0402_1005Metric, F.Cu at (103.0, 89.0)
- added RN1: R_Pack04, Resistor_SMD:R_Array_Convex_4x0603, F.Cu at (160.5, 79.5)
- added RN2: R_Pack04, Resistor_SMD:R_Array_Convex_4x0603, F.Cu at (164.5, 79.5)
- added RN3: R_Pack04, Resistor_SMD:R_Array_Convex_4x0603, F.Cu at (177.1, 92.7)
- added RN4: R_Pack04, Resistor_SMD:R_Array_Convex_4x0603, F.Cu at (177.1, 88.6)
- added U8: TPS22918DBVR, pager-jlc:SOT-23-6_L2.9-W1.6-P0.95-LS2.8-BR, F.Cu at (104.0, 86.0)
- C24: footprint Capacitor_SMD:C_0805_2012Metric -> Capacitor_SMD:C_0402_1005Metric
- C25: footprint Capacitor_SMD:C_0805_2012Metric -> Capacitor_SMD:C_0603_1608Metric
- D1: value LED -> GREEN
- D2: value LED -> BLUE
- J1: footprint Connector_PinHeader_1.27mm:PinHeader_1x05_P1.27mm_Vertical_SMD_Pin1Left -> Connector_PinHeader_1.27mm:PinHeader_1x05_P1.27mm_Vertical
- J2: footprint Connector_PinHeader_1.27mm:PinHeader_1x03_P1.27mm_Vertical_SMD_Pin1Left -> Connector_PinHeader_1.27mm:PinHeader_1x03_P1.27mm_Vertical
- R13: value 470 1% -> 470
- SW1: value SW_SPST -> B3U-1000P
- SW2: moved to F.Cu
- moved TP11 67.3 mm to (109.2, 120.8)
- moved J2 63.5 mm to (104.5, 65.5)
- moved TP4 62.0 mm to (108.0, 54.2)
- moved D1 58.8 mm to (144.0, 67.5), turned to 180 degrees
- moved D2 58.8 mm to (144.0, 70.5), turned to 180 degrees
- moved R2 57.0 mm to (144.3, 69.0), turned to 180 degrees
- moved R3 57.0 mm to (144.3, 72.0), turned to 180 degrees
- moved D4 52.5 mm to (144.0, 73.5), turned to 180 degrees
- moved R16 51.0 mm to (144.3, 75.0), turned to 0 degrees
- moved TP10 44.4 mm to (111.2, 54.2)
- moved J7 43.5 mm to (122.0, 57.5), turned to 180 degrees
- moved TP1 42.7 mm to (143.5, 84.2)
- moved C8 42.4 mm to (105.7, 83.0), turned to 0 degrees
- moved C5 42.3 mm to (106.5, 89.2), turned to -90 degrees
- moved C7 40.9 mm to (105.0, 89.5)
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Connections:
- net /input_module/TCA_KEYPAD_INT renamed /input_module/INT
- J7 pad 3: +3V3_S -> +3V3
- R8 pad 1: /mcu/IO2 -> Net-(U8-ON)
- R8 pad 2: Net-(U2-ON) -> /mcu/IO2
- TP9 pad 1: Net-(U2-ON) -> /mcu/IO2
- U7 pad 1: unconnected-(U7-ROW7-Pad1) -> Net-(RN2-R2.1)
- U7 pad 12: unconnected-(U7-COL3-Pad12) -> Net-(RN3-R1.2)
- U7 pad 13: unconnected-(U7-COL4-Pad13) -> Net-(RN3-R2.2)
- U7 pad 14: unconnected-(U7-COL5-Pad14) -> Net-(RN3-R3.2)
- U7 pad 15: unconnected-(U7-COL6-Pad15) -> Net-(RN3-R4.2)
- U7 pad 16: unconnected-(U7-COL7-Pad16) -> Net-(RN4-R1.2)
- U7 pad 17: unconnected-(U7-COL8-Pad17) -> Net-(RN4-R2.2)
- U7 pad 18: unconnected-(U7-COL9-Pad18) -> Net-(RN4-R3.2)
- U7 pad 2: unconnected-(U7-ROW6-Pad2) -> Net-(RN2-R1.1)
- U7 pad 3: unconnected-(U7-ROW5-Pad3) -> Net-(RN1-R4.1)
- U7 pad 4: unconnected-(U7-ROW4-Pad4) -> Net-(RN1-R3.1)
- U7 pad 5: unconnected-(U7-ROW3-Pad5) -> Net-(RN1-R2.1)
- U7 pad 6: unconnected-(U7-ROW2-Pad6) -> Net-(RN1-R1.1)
Routing:
- net +3V3: track 120.4 -> 38.4 mm, vias 2 -> 7
- net VDD: track 35.8 -> 97.2 mm, vias 1 -> 6
- net +3V3_S: track 97.9 -> 36.6 mm, vias 3 -> 2
- net /mcu/USB_P: track 23.1 -> 75.6 mm
- net /mcu/USB_N: track 23.1 -> 74.2 mm
- net /edp/EPD.BUSY: track 14.8 -> 58.6 mm, vias 0 -> 2
- net /mcu/NRF_RESET: track 20.3 -> 62.1 mm, vias 0 -> 1
- net +BATT: track 82.8 -> 41.9 mm
- net VDC: track 51.4 -> 13.3 mm, vias 0 -> 4
- net /input_module/INT: track 14.4 -> 49.9 mm
- net Net-(D4-A): track 57.4 -> 24.8 mm
- net /edp/EPD.CS: track 15.3 -> 46.7 mm
- net /edp/EPD.RST: track 12.4 -> 41.2 mm, vias 0 -> 2
- net +5V: track 65.0 -> 36.9 mm, vias 3 -> 7
- net /edp/EPD.DC: track 15.8 -> 42.4 mm
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- added copper zone on In2.Cu, net +3V3
- added copper zone on In2.Cu, net +3V3_S
- added copper zone on In2.Cu, net +5V
- added copper zone on In2.Cu, net +BATT
- added copper zone on In2.Cu, net VBUS
- added copper zone on In2.Cu, net VDC
Other:
- outline, holes or cut-outs redrawn
- board text added: "3V3"
- board text added: "3V3S"
- board text added: "5V"
- board text added: "BATT"
- board text added: "CELL"
- board text added: "VBUS"
- board text added: "VDC"
