File: meshpager.kicad_sch (KiCad schematic)
At the start: 0 parts

Commit message: rename project
Other:
- added sheet mcu (mcu.kicad_sch)
- title: (none) -> Meshpager
Changed lines of the file:
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@@
 	(generator_version "10.0")
 	(paper "A4")
+	(title_block
+		(title "Meshpager")
+		(date "2026-08-23")
+		(rev "1")
+	)
+	(sheet
+		(at 68.58 152.4)
+		(size 46.99 25.4)
+		(exclude_from_sim no)
+		(in_bom yes)
+		(on_board yes)
+		(dnp no)
+		(fields_autoplaced yes)
+		(stroke
+			(width 0.1524)
+			(type solid)
+		)
+		(fill
+			(color 0 0 0 0)
+		)
+		(property "Sheetname" "mcu"
+			(at 68.58 151.6884 0)
+			(show_name no)
+			(do_not_autoplace no)
+			(effects
+				(font
+					(size 1.27 1.27)
+				)
+				(justify left bottom)
+			)
+		)
+		(property "Sheetfile" "mcu.kicad_sch"
+			(at 68.58 178.3846 0)
+			(show_name no)
+			(do_not_autoplace no)
+			(effects
+				(font
+					(size 1.27 1.27)
+				)
+				(justify left top)
+			)
+		)
+		(instances
+			(project "meshpager"
+				(path "/d34a9893-cd16-421e-bfb0-6315046aba1a"
+					(page "2")
+				)
+			)
+		)
+	)
 	(sheet
 		(at 146.05 107.95)
@@
 			(project "pcb2"
 				(path "/c0ddd66c-7b46-46d3-9de5-c3245bca1945"
+					(page "4")
+				)
+			)
+			(project "meshpager"
+				(path "/d34a9893-cd16-421e-bfb0-6315046aba1a"
 					(page "4")
 				)
@@
 				)
 			)
+			(project "meshpager"
+				(path "/d34a9893-cd16-421e-bfb0-6315046aba1a"
+					(page "5")
+				)
+			)
 		)
 	)
@@
 					(page "3")
 				)
+			)
+			(project "meshpager"
+				(path "/d34a9893-cd16-421e-bfb0-6315046aba1a"
+					(page "3")
+				)

Commit message: update
Parts:
- added H1, H2, H3, H4, H5, H6: MountingHole_Pad, MountingHole:MountingHole_2.7mm_M2.5_Pad, symbol Mechanical:MountingHole_Pad
Connections:
- new net GND: H1.1, H2.1, H3.1, H4.1, H5.1, H6.1
Other:
- added sheet edp (edp.kicad_sch)
- added sheet input_module (input_module.kicad_sch)
- sheet mcu ports: added EPD.BUSY, EPD.CS, EPD.DC, EPD.MOSI, EPD.RST, EPD.SCK, I2C1.SCL, I2C1.SDA, IO2, KBD_INT, SW1, USB_N, USB_P, VBAT_ADC; removed none
- sheet power ports: added IO2, VBAT_ADC; removed none
- sheet usb-c ports: added USB_N, USB_P; removed none

Commit message: update
Parts:
- removed H5, H6: MountingHole_Pad, MountingHole:MountingHole_2.7mm_M2.5_Pad, symbol Mechanical:MountingHole_Pad
Other:
- sheet input_module ports: added none; removed SW1
- sheet mcu ports: added none; removed SW1

Commit message: Pretty cool now
Parts:
- removed H1, H2, H3, H4: MountingHole_Pad, MountingHole:MountingHole_2.7mm_M2.5_Pad, symbol Mechanical:MountingHole_Pad
- added J6, J7: HC-FPC-05-09-5RLTAG, pager-jlc:CONN-SMD_5P-P0.50_HCTL_HC-FPC-05-09-5RLTAG, symbol pager-jlc:HC-FPC-05-09-5RLTAG
Connections:
- net GND: now also J7.5, J7.6, J7.7
- net input_module/TCA_KEYPAD_INT: now also J6.1
- net input_module/TCA_SCL: now also J6.4
- net input_module/TCA_SDA: now also J6.2
- new net +3V3_S: J7.3
- new net GND1: J6.5, J6.6, J6.7
- new net VDD: J6.3
- new net mcu/I2C1.SCL: J7.4
- new net mcu/I2C1.SDA: J7.2
- new net mcu/KBD_INT: J7.1

Commit message: Update
Parts:
- added FID1, FID2, FID3, FID4, FID5, FID6: Fiducial, Fiducial:Fiducial_1mm_Mask3mm, symbol Mechanical:Fiducial
- added H5, H6, H7, H8: MountingHole_Pad, MountingHole:MountingHole_2.7mm_M2.5_Pad, symbol Mechanical:MountingHole_Pad
Connections:
- net GND: now also H5.1, H6.1, H7.1, H8.1

Commit message: Update
Parts:
- J6, J7: LCSC (none) -> C5213747
Connections:
- net +3V3_S renamed +3V3
Changed lines of the file:
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@@
+			)
+		)
+		(property "LCSC" "C5213747"
+			(at 86.36 123.19 0)
+			(hide yes)
+			(show_name no)
+			(do_not_autoplace no)
+			(effects
+				(font
+					(size 1.27 1.27)
+				)
 			)
 		)
@@
 			)
 		)
+		(property "LCSC" "C5213747"
+			(at 68.58 123.444 0)
+			(hide yes)
+			(show_name no)
+			(do_not_autoplace no)
+			(effects
+				(font
+					(size 1.27 1.27)
+				)
+			)
+		)
 		(pin "1"
 		)
@@
 			)
 		)
-		(property "Value" "+3V3_S"
+		(property "Value" "+3V3"
 			(at 95.25 123.1899 0)
 			(show_name no)
