File: power.kicad_sch (KiCad schematic)
At the start: 45 parts, among them CN1 PH-2AWT, Q1 NCE40P05Y, U1 SGM6036-3.3YUDT6G/TR, U2 SY6287CABC, U3 SGM2578AADYG/TR, U4 SGM41524YTDC8G/TR

Commit message: update
Parts:
- removed C15: 10uF, symbol Device:C
- removed C16, C18: 100nF, symbol Device:C
- removed C17: 22uF, symbol Device:C
- removed D2: RED, symbol Device:LED
- removed L2: 2.2uH, symbol Device:L_Iron
- removed R13: 15K 1%, symbol Device:R
- removed R14: 20K 1%, symbol Device:R
- removed R15: 0, symbol Device:R
- removed R16: 1K, symbol Device:R
- removed TH1: 10K, symbol Device:Thermistor_NTC
- removed U4: SGM41524YTDC8G/TR, pager-jlc:DFN-8_L3.0-W2.0-P0.50-TL-EP-1, symbol pager-jlc:SGM41524YTDC8G_TR
Connections:
- net IO2: now reaches R11.1, R12.2
Other:
- note added: "Bat Input"
- note added: "DC-DC"
- note added: "Load Switch"
- note added: "OCP"
- note added: "Power Path"
- company: Samuel Imboden -> (none)
- title: Meshpager -> (none)

Commit message: update
Parts:
- removed C2: 100uF, symbol Device:C_Polarized
- removed C6: 22pF, symbol Device:C
- removed C9: 10pF, symbol Device:C
- removed CN1: PH-2AWT, pager-jlc:CONN-SMD_PH-2AWT, symbol pager-jlc:PH-2AWT
- removed L1: 4.7uH, symbol Device:L_Iron
- removed R3: 1M 1%, symbol Device:R
- added L1: 4.7uH, pager-jlc:IND-SMD_L3.0-W3.0_FNR30XXS, symbol pager-jlc:SWPA3012S4R7MT
- added SW2: MK-12C02-G020, pager-jlc:SW-SMD_MK-12C02-G020, symbol pager-jlc:MK-12C02-G020
- added U2: GT-BTP30003-0600A-016A, pager-jlc:BAT-SMD_GT-BTP30003-0500A-016A-1, symbol pager-jlc:GT-BTP30003-0600A-016A
- C10: renamed from C7; footprint (none) -> Capacitor_SMD:C_0805_2012Metric
- C11: renamed from C8; footprint (none) -> Capacitor_SMD:C_0402_1005Metric
- C12: renamed from C13; footprint (none) -> Capacitor_SMD:C_0603_1608Metric
- C2: renamed from C14; footprint (none) -> Capacitor_SMD:C_0402_1005Metric
- C3: renamed from C1; footprint (none) -> Capacitor_SMD:C_0402_1005Metric
- C4: renamed from C3; footprint (none) -> Capacitor_SMD:C_0805_2012Metric
- C5: renamed from C10; footprint (none) -> Capacitor_SMD:C_0603_1608Metric
- C6: renamed from C4; footprint (none) -> Capacitor_SMD:C_0402_1005Metric
- C7: renamed from C11; footprint (none) -> Capacitor_SMD:C_0402_1005Metric
- C8: renamed from C5; footprint (none) -> Capacitor_SMD:C_0402_1005Metric
- C9: renamed from C12; footprint (none) -> Capacitor_SMD:C_0402_1005Metric
- R10: renamed from R2; footprint (none) -> Resistor_SMD:R_0402_1005Metric
- R11: renamed from R6; footprint (none) -> Resistor_SMD:R_0402_1005Metric
- R12: renamed from R7; footprint (none) -> Resistor_SMD:R_0402_1005Metric
- R13: renamed from R8; footprint (none) -> Resistor_SMD:R_0402_1005Metric
- R14: renamed from R9; footprint (none) -> Resistor_SMD:R_0402_1005Metric
- R4: value 806K 1% -> 1M; footprint (none) -> Resistor_SMD:R_0402_1005Metric
- R5: value 1.5M 1% -> 1.5M; footprint (none) -> Resistor_SMD:R_0402_1005Metric
- R6: renamed from R10; footprint (none) -> Resistor_SMD:R_0402_1005Metric
- R7: renamed from R11; footprint (none) -> Resistor_SMD:R_0402_1005Metric
- R8: renamed from R12; footprint (none) -> Resistor_SMD:R_0402_1005Metric
- R9: renamed from R1; footprint (none) -> Resistor_SMD:R_0402_1005Metric
- renumbered D1 to D3, U1 to U4, U2 to U5
Connections:
- net +3V3: now also U4.3 (VOUT), L1.2; no longer R5.1
- net +BATT: now also R4.1, SW2.3
- net GND: now also R5.2, SW2.4, SW2.5, SW2.6, SW2.7, U2.3 (-)
- net at U4.2 (SW): now also L1.1
- net VBAT_ADC: now reaches R4.2
- net VBAT_ADC: now also R5.1; no longer U4.3 (VOUT)
- new net BAT_CELL: SW2.1, SW2.2, U2.1 (+)
- no-connect marks 1 -> 2
Other:
- title: (none) -> Meshpager
- moved on the sheet: C10, C11, C12, C2, C3, C4, C5, C6, C7, C8, C9, D3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

Commit message: update
Parts:
- added C6: 100nF, Capacitor_SMD:C_0402_1005Metric, symbol Device:C
- added C7: 10uF, Capacitor_SMD:C_0603_1608Metric, symbol Device:C
- added C8: 1uF, Capacitor_SMD:C_0603_1608Metric, symbol Device:C
- added TP1, TP2, TP3, TP4: GND, TestPoint:TestPoint_Pad_1.5x1.5mm, symbol Connector:TestPoint
- added TP10: +3V3, TestPoint:TestPoint_Pad_1.5x1.5mm, symbol Connector:TestPoint
- added TP11: +3V3_S, TestPoint:TestPoint_Pad_1.5x1.5mm, symbol Connector:TestPoint
- added TP12: +BATT, TestPoint:TestPoint_Pad_1.5x1.5mm, symbol Connector:TestPoint
- added TP5: VBAT_ADC, TestPoint:TestPoint_Pad_1.5x1.5mm, symbol Connector:TestPoint
- added TP6: VBUS, TestPoint:TestPoint_Pad_1.5x1.5mm, symbol Connector:TestPoint
- added TP7: +5V, TestPoint:TestPoint_Pad_1.5x1.5mm, symbol Connector:TestPoint
- added TP8: VDC, TestPoint:TestPoint_Pad_1.5x1.5mm, symbol Connector:TestPoint
- added TP9: MCU_GATE, TestPoint:TestPoint_Pad_1.5x1.5mm, symbol Connector:TestPoint
- J3: renamed from U2; value GT-BTP30003-0600A-016A -> 009155003301006; footprint pager-jlc:BAT-SMD_GT-BTP30003-0500A-016A-1 -> pager:009155003301006; symbol pager-jlc:GT-BTP30003-0600A-016A -> $pager:009155003301006; Height (none) -> 6; Manufacturer_Name (none) -> Kyocera AVX; Manufacturer_Part_Number (none) -> 009155003301006; Mouser Part Number (none) -> 581-009155003301006; Mouser Price/Stock (none) -> https://www.mouser.co.uk/ProductDetail/KYOCERA-AVX/00915500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; now not fitted; now left out of the parts list
- R11: renamed from R10; value 4.7K -> 100K
- R12, R6: footprint Resistor_SMD:R_0402_1005Metric -> Resistor_SMD:R_0805_2012Metric_Pad1.20x1.40mm_HandSolder; now left out of the parts list
- R14: footprint Resistor_SMD:R_0402_1005Metric -> Resistor_SMD:R_0805_2012Metric_Pad1.20x1.40mm_HandSolder
- R9: renamed from R8; now left out of the parts list
- SW2: now not fitted
- U3: renamed from U5; Sector (none) -> OCP
- renumbered C5 to C10, C7 to C11, C4 to C12, C9 to C13, C6 to C14, C8 to C15, C10 to C16, C11 to C17, C12 to C18, C2 to C5, C3 to C9, R11 to R10, R9 to R7, R7 to R8, U3 to U2
Connections:
- net +3V3: now also C8.1, TP10.1
- net +3V3_S: now also C7.1, TP11.1
- net +5V: now also TP7.1
- net +BATT: now also TP12.1
- net BAT_CELL: now also J3.5 (+); no longer J3.1 (+)
- net GND: now also J3.1 (-), C6.2, C7.2, C8.2, TP1.1, TP2.1, TP3.1, TP4.1; no longer J3.3 (-)
- net VBAT_ADC: now also C6.1, TP5.1
- net VBUS: now also TP6.1
- net VDC: now also TP8.1
- net at R8.2, U2.B2 (ON): now also TP9.1
Other:
- note added: "Testpoints"
- moved on the sheet: C12, C14, C15, C16, C17, C5, L1, R11, R6, R8, R9, U2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

Commit message: Update
Parts:
- TP1, TP10, TP11, TP12, TP2, TP3, TP4, TP5, TP6, TP7, TP8, TP9: footprint TestPoint:TestPoint_Pad_1.5x1.5mm -> TestPoint:TestPoint_Pad_D1.5mm; now left out of the parts list
Changed lines of the file:
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@@
 		(body_style 1)
 		(exclude_from_sim no)
-		(in_bom yes)
+		(in_bom no)
 		(on_board yes)
 		(in_pos_files yes)
@@
 			)
 		)
-		(property "Footprint" "TestPoint:TestPoint_Pad_1.5x1.5mm"
+		(property "Footprint" "TestPoint:TestPoint_Pad_D1.5mm"
 			(at 21.59 184.15 0)
 			(hide yes)
@@
 		(body_style 1)
 		(exclude_from_sim no)
-		(in_bom yes)
+		(in_bom no)
 		(on_board yes)
 		(in_pos_files yes)
@@
 			)
 		)
-		(property "Footprint" "TestPoint:TestPoint_Pad_1.5x1.5mm"
+		(property "Footprint" "TestPoint:TestPoint_Pad_D1.5mm"
 			(at 91.44 177.8 0)
 			(hide yes)
@@
 		(body_style 1)
 		(exclude_from_sim no)
-		(in_bom yes)
+		(in_bom no)
 		(on_board yes)
 		(in_pos_files yes)
@@
 			)
 		)
-		(property "Footprint" "TestPoint:TestPoint_Pad_1.5x1.5mm"
+		(property "Footprint" "TestPoint:TestPoint_Pad_D1.5mm"
 			(at 30.48 168.91 0)
 			(hide yes)
@@
 		(body_style 1)
 		(exclude_from_sim no)
-		(in_bom yes)
+		(in_bom no)
 		(on_board yes)
 		(in_pos_files yes)
@@
 			)
 		)
-		(property "Footprint" "TestPoint:TestPoint_Pad_1.5x1.5mm"
+		(property "Footprint" "TestPoint:TestPoint_Pad_D1.5mm"
 			(at 34.29 60.96 0)
 			(hide yes)
@@
 		(body_style 1)
 		(exclude_from_sim no)
-		(in_bom yes)
+		(in_bom no)
 		(on_board yes)
 		(in_pos_files yes)
@@
 			)
 		)
-		(property "Footprint" "TestPoint:TestPoint_Pad_1.5x1.5mm"
+		(property "Footprint" "TestPoint:TestPoint_Pad_D1.5mm"
 			(at 105.41 177.8 0)
 			(hide yes)
@@
 		(body_style 1)
 		(exclude_from_sim no)
-		(in_bom yes)
+		(in_bom no)
 		(on_board yes)
 		(in_pos_files yes)
@@
 			)
 		)
-		(property "Footprint" "TestPoint:TestPoint_Pad_1.5x1.5mm"
+		(property "Footprint" "TestPoint:TestPoint_Pad_D1.5mm"
 			(at 99.06 99.06 0)
 			(hide yes)
@@
 		(body_style 1)
 		(exclude_from_sim no)
-		(in_bom yes)
+		(in_bom no)
 		(on_board yes)
 		(in_pos_files yes)
@@
 			)
 		)
-		(property "Footprint" "TestPoint:TestPoint_Pad_1.5x1.5mm"
+		(property "Footprint" "TestPoint:TestPoint_Pad_D1.5mm"
 			(at 49.53 177.8 0)
 			(hide yes)
@@
 		(body_style 1)
 		(exclude_from_sim no)
-		(in_bom yes)
+		(in_bom no)
 		(on_board yes)
 		(in_pos_files yes)
@@
 			)
 		)
-		(property "Footprint" "TestPoint:TestPoint_Pad_1.5x1.5mm"
+		(property "Footprint" "TestPoint:TestPoint_Pad_D1.5mm"
 			(at 30.48 184.15 0)
 			(hide yes)
@@
 		(body_style 1)
 		(exclude_from_sim no)
-		(in_bom yes)
+		(in_bom no)
 		(on_board yes)
 		(in_pos_files yes)
@@
 			)
 		)
-		(property "Footprint" "TestPoint:TestPoint_Pad_1.5x1.5mm"
+		(property "Footprint" "TestPoint:TestPoint_Pad_D1.5mm"
 			(at 77.47 177.8 0)
 			(hide yes)
@@
 		(body_style 1)
 		(exclude_from_sim no)
-		(in_bom yes)
+		(in_bom no)
 		(on_board yes)
 		(in_pos_files yes)
@@
 			)
 		)
-		(property "Footprint" "TestPoint:TestPoint_Pad_1.5x1.5mm"
+		(property "Footprint" "TestPoint:TestPoint_Pad_D1.5mm"
 			(at 63.5 177.8 0)
 			(hide yes)
@@
 		(body_style 1)
 		(exclude_from_sim no)
-		(in_bom yes)
+		(in_bom no)
 		(on_board yes)
 		(in_pos_files yes)
@@
 			)
 		)
-		(property "Footprint" "TestPoint:TestPoint_Pad_1.5x1.5mm"
+		(property "Footprint" "TestPoint:TestPoint_Pad_D1.5mm"
 			(at 119.38 177.8 0)
 			(hide yes)
@@
 		(body_style 1)
 		(exclude_from_sim no)
-		(in_bom yes)
+		(in_bom no)
 		(on_board yes)
 		(in_pos_files yes)
@@
 			)
 		)
-		(property "Footprint" "TestPoint:TestPoint_Pad_1.5x1.5mm"
+		(property "Footprint" "TestPoint:TestPoint_Pad_D1.5mm"
 			(at 21.59 168.91 0)
 			(hide yes)

Commit message: Pretty cool now
Parts:
- removed TP3: GND, TestPoint:TestPoint_Pad_D1.5mm, symbol Connector:TestPoint
Changed lines of the file:
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@@
 	(wire
 		(pts
-			(xy 25.4 168.91) (xy 25.4 171.45)
-		)
-		(stroke
-			(width 0)
-			(type default)
-		)
-	)
-	(wire
-		(pts
 			(xy 100.33 54.61) (xy 100.33 49.53)
 		)
@@
 	)
 	(symbol
-		(lib_id "Connector:TestPoint")
-		(at 25.4 168.91 0)
-		(unit 1)
-		(body_style 1)
-		(exclude_from_sim no)
-		(in_bom no)
-		(on_board yes)
-		(in_pos_files yes)
-		(dnp no)
-		(fields_autoplaced yes)
-		(property "Reference" "TP3"
-			(at 27.94 164.3379 0)
-			(show_name no)
-			(do_not_autoplace no)
-			(effects
-				(font
-					(size 1.27 1.27)
-				)
-				(justify left)
-			)
-		)
-		(property "Value" "GND"
-			(at 27.94 166.8779 0)
-			(show_name no)
-			(do_not_autoplace no)
-			(effects
-				(font
-					(size 1.27 1.27)
-				)
-				(justify left)
-			)
-		)
-		(property "Footprint" "TestPoint:TestPoint_Pad_D1.5mm"
-			(at 30.48 168.91 0)
-			(hide yes)
-			(show_name no)
-			(do_not_autoplace no)
-			(effects
-				(font
-					(size 1.27 1.27)
-				)
-			)
-		)
-		(property "Datasheet" ""
-			(at 30.48 168.91 0)
-			(hide yes)
-			(show_name no)
-			(do_not_autoplace no)
-			(effects
-				(font
-					(size 1.27 1.27)
-				)
-			)
-		)
-		(property "Description" "test point"
-			(at 25.4 168.91 0)
-			(hide yes)
-			(show_name no)
-			(do_not_autoplace no)
-			(effects
-				(font
-					(size 1.27 1.27)
-				)
-			)
-		)
-		(pin "1"
-		)
-		(instances
-			(project "meshpager"
-				(path "/d34a9893-cd16-421e-bfb0-6315046aba1a/c31e5c72-3f65-4932-a34e-bb5f91e41816"
-					(reference "TP3")
-					(unit 1)
-				)
-			)
-		)
-	)
-	(symbol
 		(lib_id "Device:C")
 		(at 236.22 134.62 180)
@@
 					(unit 1)
 				)
-			)
-		)
-	)
-	(symbol
-		(lib_id "power:GND")
-		(at 25.4 171.45 0)
-		(unit 1)
-		(body_style 1)
-		(exclude_from_sim no)
-		(in_bom yes)
-		(on_board yes)
-		(in_pos_files yes)
-		(dnp no)
-		(fields_autoplaced yes)
-		(property "Reference" "#PWR019"
-			(at 25.4 177.8 0)
-			(hide yes)
-			(show_name no)
-			(do_not_autoplace no)
-			(effects
-				(font
-					(size 1.27 1.27)
-				)
-			)
-		)
-		(property "Value" "GND"
-			(at 25.4 176.53 0)
-			(show_name no)
-			(do_not_autoplace no)
-			(effects
-				(font
-					(size 1.27 1.27)
-				)
-			)
-		)
-		(property "Footprint" ""
-			(at 25.4 171.45 0)
-			(hide yes)
-			(show_name no)
-			(do_not_autoplace no)
-			(effects
-				(font
-					(size 1.27 1.27)
-				)
-			)
-		)
-		(property "Datasheet" ""
-			(at 25.4 171.45 0)
-			(hide yes)
-			(show_name no)
-			(do_not_autoplace no)
-			(effects
-				(font
-					(size 1.27 1.27)
-				)
-			)
-		)
-		(property "Description" "Power symbol creates a global label with name \"GND\" , ground"
-			(at 25.4 171.45 0)
-			(hide yes)
-			(show_name no)
-			(do_not_autoplace no)
-			(effects
-				(font
-					(size 1.27 1.27)
-				)
-			)
-		)
-		(pin "1"
-		)
-		(instances
-			(project "meshpager"
-				(path "/d34a9893-cd16-421e-bfb0-6315046aba1a/c31e5c72-3f65-4932-a34e-bb5f91e41816"
-					(reference "#PWR019")
-					(unit 1)
-				)

Commit message: Update
Parts:
- removed R6: 0, Resistor_SMD:R_0805_2012Metric_Pad1.20x1.40mm_HandSolder, symbol Device:R
- removed U2: SGM2578AADYG/TR, pager-jlc:WLCSP-4_L0.9-W0.9-R2-C2-P0.50-TL, symbol pager-jlc:SGM2578AADYG_TR
- added C26: 1nF, Capacitor_SMD:C_0402_1005Metric, symbol Device:C
- added U8: TPS22918DBVR, pager-jlc:SOT-23-6_L2.9-W1.6-P0.95-LS2.8-BR, symbol pager-jlc:TPS22918DBVR
- C10, C18, C7: LCSC (none) -> C19702
- C11, C13, C14, C15, C17, C5, C6, C9: LCSC (none) -> C1525
- C12, C16: LCSC (none) -> C45783
- C8: LCSC (none) -> C15849
- D3: LCSC (none) -> C43381
- J3: LCSC (none) -> C41378740; LCSC Part C41378740 -> (none); MPN GT-BTP30003-0600A-016A -> (none); Manufacturer G-Switch(品赞) -> (none); now in the parts list
- L1: LCSC (none) -> C83415
- Q1: LCSC (none) -> C163738
- R10, R11: LCSC (none) -> C25741
- R12, R14: LCSC (none) -> C17477
- R13: LCSC (none) -> C25117
- R4: LCSC (none) -> C26083
- R5: LCSC (none) -> C22276
- R7: LCSC (none) -> C25900
- R8: LCSC (none) -> C25744
- R9: LCSC (none) -> C25741; now fitted; now in the parts list
- SW2: LCSC (none) -> C963206; now fitted
- U3: LCSC (none) -> C3013652
- U4: LCSC (none) -> C5153601
Connections:
- net +3V3: now also U8.1 (VIN)
- net +3V3_S: now also U8.5 (QOD), U8.6 (VOUT)
- net GND: now also C26.2, U8.2 (GND)
- net IO2: now also R8.2, TP9.1; no longer R8.1
- new net: C26.1, U8.4 (CT)
- new net: R8.1, U8.3 (ON)
- no-connect marks 2 -> 3
Other:
- moved on the sheet: C5, C7, C8, R8, TP9
