File: usb-c.kicad_sch (KiCad schematic)
At the start: 4 parts, among them J2 USB_C_Receptacle_USB2.0_16P, U5 USBLC6-2SC6

Commit message: update
Parts:
- R18: renamed from R17; footprint (none) -> Resistor_SMD:R_0402_1005Metric
- R19: renamed from R18; footprint (none) -> Resistor_SMD:R_0402_1005Metric
- renumbered U5 to U7
Other:
- title: (none) -> Meshpager
Changed lines of the file:
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@@
 	(generator_version "10.0")
 	(paper "A4")
+	(title_block
+		(title "Meshpager")
+		(date "2026-08-23")
+		(rev "1")
+	)
 	(junction
 		(at 138.43 102.87)
@@
 		(dnp no)
 		(fields_autoplaced yes)
-		(property "Reference" "#PWR023"
+		(property "Reference" "#PWR044"
 			(at 138.43 85.09 0)
 			(hide yes)
@@
 				(path "/c0ddd66c-7b46-46d3-9de5-c3245bca1945/b97176e7-7611-493e-95a1-ff46bfacccdf"
 					(reference "#PWR023")
+					(unit 1)
+				)
+			)
+			(project "meshpager"
+				(path "/d34a9893-cd16-421e-bfb0-6315046aba1a/b97176e7-7611-493e-95a1-ff46bfacccdf"
+					(reference "#PWR044")
 					(unit 1)
 				)
@@
 		(dnp no)
 		(fields_autoplaced yes)
-		(property "Reference" "#PWR034"
+		(property "Reference" "#PWR045"
 			(at 161.29 93.98 0)
 			(hide yes)
@@
 				(path "/c0ddd66c-7b46-46d3-9de5-c3245bca1945/b97176e7-7611-493e-95a1-ff46bfacccdf"
 					(reference "#PWR034")
+					(unit 1)
+				)
+			)
+			(project "meshpager"
+				(path "/d34a9893-cd16-421e-bfb0-6315046aba1a/b97176e7-7611-493e-95a1-ff46bfacccdf"
+					(reference "#PWR045")
 					(unit 1)
 				)
@@
 		(dnp no)
 		(fields_autoplaced yes)
-		(property "Reference" "#PWR036"
+		(property "Reference" "#PWR046"
 			(at 168.91 95.25 0)
 			(hide yes)
@@
 				(path "/c0ddd66c-7b46-46d3-9de5-c3245bca1945/b97176e7-7611-493e-95a1-ff46bfacccdf"
 					(reference "#PWR036")
+					(unit 1)
+				)
+			)
+			(project "meshpager"
+				(path "/d34a9893-cd16-421e-bfb0-6315046aba1a/b97176e7-7611-493e-95a1-ff46bfacccdf"
+					(reference "#PWR046")
 					(unit 1)
 				)
@@
 				)
 			)
+			(project "meshpager"
+				(path "/d34a9893-cd16-421e-bfb0-6315046aba1a/b97176e7-7611-493e-95a1-ff46bfacccdf"
+					(reference "J2")
+					(unit 1)
+				)
+			)
 		)
 	)
@@
 		(in_pos_files yes)
 		(dnp no)
-		(property "Reference" "R18"
+		(property "Reference" "R19"
 			(at 146.05 97.536 90)
 			(show_name no)
@@
 			)
 		)
-		(property "Footprint" ""
+		(property "Footprint" "Resistor_SMD:R_0402_1005Metric"
 			(at 146.05 97.028 90)
 			(hide yes)
@@
 				(path "/c0ddd66c-7b46-46d3-9de5-c3245bca1945/b97176e7-7611-493e-95a1-ff46bfacccdf"
 					(reference "R18")
+					(unit 1)
+				)
+			)
+			(project "meshpager"
+				(path "/d34a9893-cd16-421e-bfb0-6315046aba1a/b97176e7-7611-493e-95a1-ff46bfacccdf"
+					(reference "R19")
 					(unit 1)
 				)
@@
 		(dnp no)
 		(fields_autoplaced yes)
-		(property "Reference" "#PWR035"
+		(property "Reference" "#PWR047"
 			(at 168.91 121.92 0)
 			(hide yes)
@@
 				(path "/c0ddd66c-7b46-46d3-9de5-c3245bca1945/b97176e7-7611-493e-95a1-ff46bfacccdf"
 					(reference "#PWR035")
+					(unit 1)
+				)
+			)
+			(project "meshpager"
+				(path "/d34a9893-cd16-421e-bfb0-6315046aba1a/b97176e7-7611-493e-95a1-ff46bfacccdf"
+					(reference "#PWR047")
 					(unit 1)
 				)
@@
 		(dnp no)
 		(fields_autoplaced yes)
-		(property "Reference" "#PWR013"
+		(property "Reference" "#PWR043"
 			(at 119.38 135.89 0)
 			(hide yes)
@@
 				(path "/c0ddd66c-7b46-46d3-9de5-c3245bca1945/b97176e7-7611-493e-95a1-ff46bfacccdf"
 					(reference "#PWR013")
+					(unit 1)
+				)
+			)
+			(project "meshpager"
+				(path "/d34a9893-cd16-421e-bfb0-6315046aba1a/b97176e7-7611-493e-95a1-ff46bfacccdf"
+					(reference "#PWR043")
 					(unit 1)
 				)
@@
 		(dnp no)
 		(fields_autoplaced yes)
-		(property "Reference" "U5"
+		(property "Reference" "U7"
 			(at 170.5611 95.25 0)
 			(show_name no)
@@
 				(path "/c0ddd66c-7b46-46d3-9de5-c3245bca1945/b97176e7-7611-493e-95a1-ff46bfacccdf"
 					(reference "U5")
+					(unit 1)
+				)
+			)
+			(project "meshpager"
+				(path "/d34a9893-cd16-421e-bfb0-6315046aba1a/b97176e7-7611-493e-95a1-ff46bfacccdf"
+					(reference "U7")
 					(unit 1)
 				)
@@
 		(in_pos_files yes)
 		(dnp no)
-		(property "Reference" "R17"
+		(property "Reference" "R18"
 			(at 146.05 90.678 90)
 			(show_name no)
@@
 			)
 		)
-		(property "Footprint" ""
+		(property "Footprint" "Resistor_SMD:R_0402_1005Metric"
 			(at 146.05 94.488 90)
 			(hide yes)
@@
 					(unit 1)
 				)
+			)
+			(project "meshpager"
+				(path "/d34a9893-cd16-421e-bfb0-6315046aba1a/b97176e7-7611-493e-95a1-ff46bfacccdf"
+					(reference "R18")
+					(unit 1)
+				)

Commit message: update
Parts:
- removed J2: USB_C_Receptacle_USB2.0_16P, Connector_USB:USB_C_Receptacle_HRO_TYPE-C-31-M-12, symbol Connector:USB_C_Receptacle_USB2.0_16P
- added J4: USB_C_Receptacle_USB2.0_16P, Connector_USB:USB_C_Receptacle_G-Switch_GT-USB-7010ASV, symbol Connector:USB_C_Receptacle_USB2.0_16P
- renumbered U7 to U6
Connections:
- net GND: now also J4.A1 (GND), J4.A12 (GND), J4.B1 (GND), J4.B12 (GND), J4.SH (SHIELD)
- net VBUS: now also J4.A4 (VBUS), J4.A9 (VBUS), J4.B4 (VBUS), J4.B9 (VBUS)
- net at R18.1: now also J4.A5 (CC1)
- net at U6.3 (I/O2): now also J4.A6 (D+), J4.B6 (D+)
- net at U6.1 (I/O1): now also J4.A7 (D-), J4.B7 (D-)
- net at R19.1: now also J4.B5 (CC2)
Changed lines of the file:
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@@
+	)
+	(junction
+		(at 138.43 105.41)
+		(diameter 0)
+		(color 0 0 0 0)
 	)
 	(junction
 		(at 119.38 128.27)
-		(diameter 0)
-		(color 0 0 0 0)
-	)
-	(junction
-		(at 138.43 105.41)
 		(diameter 0)
 		(color 0 0 0 0)
@@
 			)
 			(justify left)
+		)
+	)
+	(symbol
+		(lib_id "Connector:USB_C_Receptacle_USB2.0_16P")
+		(at 123.19 102.87 0)
+		(unit 1)
+		(body_style 1)
+		(exclude_from_sim no)
+		(in_bom yes)
+		(on_board yes)
+		(in_pos_files yes)
+		(dnp no)
+		(fields_autoplaced yes)
+		(property "Reference" "J4"
+			(at 123.19 80.01 0)
+			(show_name no)
+			(do_not_autoplace no)
+			(effects
+				(font
+					(size 1.27 1.27)
+				)
+			)
+		)
+		(property "Value" "USB_C_Receptacle_USB2.0_16P"
+			(at 123.19 82.55 0)
+			(show_name no)
+			(do_not_autoplace no)
+			(effects
+				(font
+					(size 1.27 1.27)
+				)
+			)
+		)
+		(property "Footprint" "Connector_USB:USB_C_Receptacle_G-Switch_GT-USB-7010ASV"
+			(at 127 102.87 0)
+			(hide yes)
+			(show_name no)
+			(do_not_autoplace no)
+			(effects
+				(font
+					(size 1.27 1.27)
+				)
+			)
+		)
+		(property "Datasheet" "https://www.usb.org/sites/default/files/documents/usb_type-c.zip"
+			(at 127 102.87 0)
+			(hide yes)
+			(show_name no)
+			(do_not_autoplace no)
+			(effects
+				(font
+					(size 1.27 1.27)
+				)
+			)
+		)
+		(property "Description" "USB 2.0-only 16P Type-C Receptacle connector"
+			(at 123.19 102.87 0)
+			(hide yes)
+			(show_name no)
+			(do_not_autoplace no)
+			(effects
+				(font
+					(size 1.27 1.27)
+				)
+			)
+		)
+		(property "LCSC Part" "C2988369"
+			(at 123.19 102.87 0)
+			(hide yes)
+			(show_name no)
+			(do_not_autoplace no)
+			(effects
+				(font
+					(size 1.27 1.27)
+				)
+			)
+		)
+		(pin "A12"
+		)
+		(pin "A6"
+		)
+		(pin "A4"
+		)
+		(pin "B8"
+		)
+		(pin "B12"
+		)
+		(pin "B1"
+		)
+		(pin "B5"
+		)
+		(pin "B6"
+		)
+		(pin "A1"
+		)
+		(pin "A7"
+		)
+		(pin "A8"
+		)
+		(pin "A9"
+		)
+		(pin "A5"
+		)
+		(pin "B7"
+		)
+		(pin "SH"
+		)
+		(pin "B9"
+		)
+		(pin "B4"
+		)
+		(instances
+			(project "meshpager"
+				(path "/d34a9893-cd16-421e-bfb0-6315046aba1a/b97176e7-7611-493e-95a1-ff46bfacccdf"
+					(reference "J4")
+					(unit 1)
+				)
+			)
 		)
 	)
@@
 		(dnp no)
 		(fields_autoplaced yes)
-		(property "Reference" "#PWR044"
+		(property "Reference" "#PWR055"
 			(at 138.43 85.09 0)
 			(hide yes)
@@
 		)
 		(property "Value" "VBUS"
-			(at 138.43 76.2 0)
-			(show_name no)
-			(do_not_autoplace no)
-			(effects
-				(font
-					(size 1.27 1.27)
-				)
+			(at 140.97 80.0099 0)
+			(show_name no)
+			(do_not_autoplace no)
+			(effects
+				(font
+					(size 1.27 1.27)
+				)
+				(justify left)
 			)
 		)
@@
 			(project "meshpager"
 				(path "/d34a9893-cd16-421e-bfb0-6315046aba1a/b97176e7-7611-493e-95a1-ff46bfacccdf"
-					(reference "#PWR044")
+					(reference "#PWR055")
 					(unit 1)
 				)
@@
 		(dnp no)
 		(fields_autoplaced yes)
-		(property "Reference" "#PWR045"
+		(property "Reference" "#PWR056"
 			(at 161.29 93.98 0)
 			(hide yes)
@@
 			(project "meshpager"
 				(path "/d34a9893-cd16-421e-bfb0-6315046aba1a/b97176e7-7611-493e-95a1-ff46bfacccdf"
-					(reference "#PWR045")
+					(reference "#PWR056")
 					(unit 1)
 				)
@@
 		(dnp no)
 		(fields_autoplaced yes)
-		(property "Reference" "#PWR046"
+		(property "Reference" "#PWR057"
 			(at 168.91 95.25 0)
 			(hide yes)
@@
 		)
 		(property "Value" "VBUS"
-			(at 168.91 86.36 0)
-			(show_name no)
-			(do_not_autoplace no)
-			(effects
-				(font
-					(size 1.27 1.27)
-				)
+			(at 171.45 90.1699 0)
+			(show_name no)
+			(do_not_autoplace no)
+			(effects
+				(font
+					(size 1.27 1.27)
+				)
+				(justify left)
 			)
 		)
@@
 			(project "meshpager"
 				(path "/d34a9893-cd16-421e-bfb0-6315046aba1a/b97176e7-7611-493e-95a1-ff46bfacccdf"
-					(reference "#PWR046")
-					(unit 1)
-				)
-			)
-		)
-	)
-	(symbol
-		(lib_id "Connector:USB_C_Receptacle_USB2.0_16P")
-		(at 123.19 102.87 0)
-		(unit 1)
-		(body_style 1)
-		(exclude_from_sim no)
-		(in_bom yes)
-		(on_board yes)
-		(in_pos_files yes)
-		(dnp no)
-		(fields_autoplaced yes)
-		(property "Reference" "J2"
-			(at 123.19 80.01 0)
-			(show_name no)
-			(do_not_autoplace no)
-			(effects
-				(font
-					(size 1.27 1.27)
-				)
-			)
-		)
-		(property "Value" "USB_C_Receptacle_USB2.0_16P"
-			(at 123.19 82.55 0)
-			(show_name no)
-			(do_not_autoplace no)
-			(effects
-				(font
-					(size 1.27 1.27)
-				)
-			)
-		)
-		(property "Footprint" "Connector_USB:USB_C_Receptacle_HRO_TYPE-C-31-M-12"
-			(at 127 102.87 0)
-			(hide yes)
-			(show_name no)
-			(do_not_autoplace no)
-			(effects
-				(font
-					(size 1.27 1.27)
-				)
-			)
-		)
-		(property "Datasheet" "https://www.usb.org/sites/default/files/documents/usb_type-c.zip"
-			(at 127 102.87 0)
-			(hide yes)
-			(show_name no)
-			(do_not_autoplace no)
-			(effects
-				(font
-					(size 1.27 1.27)
-				)
-			)
-		)
-		(property "Description" "USB 2.0-only 16P Type-C Receptacle connector"
-			(at 123.19 102.87 0)
-			(hide yes)
-			(show_name no)
-			(do_not_autoplace no)
-			(effects
-				(font
-					(size 1.27 1.27)
-				)
-			)
-		)
-		(pin "A9"
-		)
-		(pin "A12"
-		)
-		(pin "B6"
-		)
-		(pin "A7"
-		)
-		(pin "B9"
-		)
-		(pin "SH"
-		)
-		(pin "A5"
-		)
-		(pin "B5"
-		)
-		(pin "A1"
-		)
-		(pin "A4"
-		)
-		(pin "A6"
-		)
-		(pin "A8"
-		)
-		(pin "B1"
-		)
-		(pin "B4"
-		)
-		(pin "B7"
-		)
-		(pin "B8"
-		)
-		(pin "B12"
-		)
-		(instances
-			(project "pcb2"
-				(path "/c0ddd66c-7b46-46d3-9de5-c3245bca1945/b97176e7-7611-493e-95a1-ff46bfacccdf"
-					(reference "J2")
-					(unit 1)
-				)
-			)
-			(project "meshpager"
-				(path "/d34a9893-cd16-421e-bfb0-6315046aba1a/b97176e7-7611-493e-95a1-ff46bfacccdf"
-					(reference "J2")
+					(reference "#PWR057")
 					(unit 1)
 				)
@@
 		(in_pos_files yes)
 		(dnp no)
+		(fields_autoplaced yes)
 		(property "Reference" "R19"
-			(at 146.05 97.536 90)
+			(at 146.05 99.06 90)
 			(show_name no)
 			(do_not_autoplace no)
@@
 		)
 		(property "Value" "5.1K"
-			(at 146.05 95.25 90)
+			(at 146.05 101.6 90)
 			(show_name no)
 			(do_not_autoplace no)
@@
 		(dnp no)
 		(fields_autoplaced yes)
-		(property "Reference" "#PWR047"
+		(property "Reference" "#PWR058"
 			(at 168.91 121.92 0)
 			(hide yes)
@@
 		)
 		(property "Value" "GND"
-			(at 168.91 120.65 0)
-			(show_name no)
-			(do_not_autoplace no)
-			(effects
-				(font
-					(size 1.27 1.27)
-				)
+			(at 171.45 116.8399 0)
+			(show_name no)
+			(do_not_autoplace no)
+			(effects
+				(font
+					(size 1.27 1.27)
+				)
+				(justify left)
 			)
 		)
@@
 			(project "meshpager"
 				(path "/d34a9893-cd16-421e-bfb0-6315046aba1a/b97176e7-7611-493e-95a1-ff46bfacccdf"
-					(reference "#PWR047")
+					(reference "#PWR058")
 					(unit 1)
 				)
@@
 		(dnp no)
 		(fields_autoplaced yes)
-		(property "Reference" "#PWR043"
+		(property "Reference" "#PWR054"
 			(at 119.38 135.89 0)
 			(hide yes)
@@
 		)
 		(property "Value" "GND"
-			(at 119.38 134.62 0)
-			(show_name no)
-			(do_not_autoplace no)
-			(effects
-				(font
-					(size 1.27 1.27)
-				)
+			(at 121.92 130.8099 0)
+			(show_name no)
+			(do_not_autoplace no)
+			(effects
+				(font
+					(size 1.27 1.27)
+				)
+				(justify left)
 			)
 		)
@@
 			(project "meshpager"
 				(path "/d34a9893-cd16-421e-bfb0-6315046aba1a/b97176e7-7611-493e-95a1-ff46bfacccdf"
-					(reference "#PWR043")
+					(reference "#PWR054")
 					(unit 1)
 				)
@@
 		(dnp no)
 		(fields_autoplaced yes)
-		(property "Reference" "U7"
+		(property "Reference" "U6"
 			(at 170.5611 95.25 0)
 			(show_name no)
@@
 			(project "meshpager"
 				(path "/d34a9893-cd16-421e-bfb0-6315046aba1a/b97176e7-7611-493e-95a1-ff46bfacccdf"
-					(reference "U7")
+					(reference "U6")
 					(unit 1)
 				)
@@
 		(in_pos_files yes)
 		(dnp no)
+		(fields_autoplaced yes)
 		(property "Reference" "R18"
-			(at 146.05 90.678 90)
+			(at 146.05 86.36 90)
 			(show_name no)
 			(do_not_autoplace no)
@@
 		)
 		(property "Value" "5.1K"
-			(at 146.05 92.71 90)
-			(show_name no)
-			(do_not_autoplace no)
+			(at 146.05 88.9 90)
+			(show_name no)
+			(do_not_autoplace no)

Commit message: Update
Parts:
- J4: LCSC (none) -> C2988369
- R18, R19: LCSC (none) -> C25905
- U6: LCSC (none) -> C7519
Changed lines of the file:
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@@
+			)
+		)
+		(property "LCSC" "C2988369"
+			(at 123.19 80.01 0)
+			(hide yes)
+			(show_name no)
+			(do_not_autoplace no)
+			(effects
+				(font
+					(size 1.27 1.27)
+				)
 			)
 		)
@@
 			)
 		)
+		(property "LCSC" "C25905"
+			(at 146.05 99.06 0)
+			(hide yes)
+			(show_name no)
+			(do_not_autoplace no)
+			(effects
+				(font
+					(size 1.27 1.27)
+				)
+			)
+		)
 		(pin "2"
 		)
@@
 			)
 		)
+		(property "LCSC" "C7519"
+			(at 170.5611 95.25 0)
+			(hide yes)
+			(show_name no)
+			(do_not_autoplace no)
+			(effects
+				(font
+					(size 1.27 1.27)
+				)
+			)
+		)
 		(pin "3"
 		)
@@
 			(hide yes)
 			(show_name no)
+			(do_not_autoplace no)
+			(effects
+				(font
+					(size 1.27 1.27)
+				)
+			)
+		)
+		(property "LCSC" "C25905"
+			(at 146.05 86.36 0)
+			(hide yes)
+			(show_name no)
